File: untitled.brd (EAGLE design)
At the start: 100 x 80 mm, 1 part

Commit message: add
Parts:
- moved U$1 78.1 mm to (76.5, 34.8), turned to 90 degrees
Other:
- board size 100 x 80 mm -> 100 x 70 mm
Changed lines of the file:
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@@
 <setting verticaltext="up"/>
 </settings>
-<grid distance="50" unitdist="mil" unit="mil" style="lines" multiple="1" display="no" altdistance="5" altunitdist="mil" altunit="mil"/>
+<grid distance="10" unitdist="mm" unit="mm" style="lines" multiple="1" display="yes" altdistance="5" altunitdist="mil" altunit="mil"/>
 <layers>
 <layer number="1" name="Top" color="4" fill="1" visible="yes" active="yes"/>
@@
 <layer number="43" name="vRestrict" color="2" fill="10" visible="yes" active="yes"/>
 <layer number="44" name="Drills" color="7" fill="1" visible="no" active="yes"/>
-<layer number="45" name="Holes" color="7" fill="1" visible="no" active="yes"/>
-<layer number="46" name="Milling" color="3" fill="1" visible="no" active="yes"/>
+<layer number="45" name="Holes" color="7" fill="1" visible="yes" active="yes"/>
+<layer number="46" name="Milling" color="3" fill="1" visible="yes" active="yes"/>
 <layer number="47" name="Measures" color="7" fill="1" visible="no" active="yes"/>
 <layer number="48" name="Document" color="7" fill="1" visible="yes" active="yes"/>
@@
 <plain>
 <wire x1="0" y1="0" x2="100" y2="0" width="0" layer="20"/>
-<wire x1="100" y1="0" x2="100" y2="80" width="0" layer="20"/>
-<wire x1="100" y1="80" x2="0" y2="80" width="0" layer="20"/>
-<wire x1="0" y1="80" x2="0" y2="0" width="0" layer="20"/>
+<wire x1="100" y1="0" x2="100" y2="70" width="0" layer="20"/>
+<wire x1="100" y1="70" x2="0" y2="70" width="0" layer="20"/>
+<wire x1="0" y1="70" x2="0" y2="40" width="0" layer="20"/>
+<wire x1="0" y1="40" x2="40" y2="40" width="0" layer="20"/>
+<wire x1="40" y1="40" x2="40" y2="30" width="0" layer="20"/>
+<wire x1="40" y1="30" x2="0" y2="30" width="0" layer="20"/>
+<wire x1="0" y1="30" x2="0" y2="0" width="0" layer="20"/>
 </plain>
 <attributes>
@@
 </autorouter>
 <elements>
-<element name="U$1" library="untitled" package="EE40/EI40" value="TRANSFORMER-EE40" x="16.51" y="-15.24" smashed="yes"/>
+<element name="U$1" library="untitled" package="EE40/EI40" value="TRANSFORMER-EE40" x="76.51" y="34.76" smashed="yes" rot="R90"/>
 </elements>
 <signals>

Commit message: add
Parts:
- removed U$1: TRANSFORMER-EE40, untitled:EE40/EI40
- added U$2: TRANSFORMER-EE40-DOWN, untitled:EE40/EI40-DOWN
Changed lines of the file:
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@@
 </autorouter>
 <elements>
-<element name="U$1" library="untitled" package="EE40/EI40" value="TRANSFORMER-EE40" x="76.51" y="34.76" smashed="yes" rot="R90"/>
+<element name="U$2" library="untitled" package="EE40/EI40-DOWN" value="TRANSFORMER-EE40-DOWN" x="73.208" y="36.477" smashed="yes"/>
 </elements>
 <signals>

Commit message: add
Parts:
- added B1: (no value), rectifier:GBU4S
- added C1: (no value), capacitor-wima:C10B4
- added C2: (no value), capacitor-wima:C2.5-2
- added GND, VCC: MOUNT-PAD-SQUARE5.0, holes:5,0-PAD-SQUARE
- added IC1: TL494CD, linear:SO16
- added Q1, Q2: IRF740, transistor-power:TO220BV
- added R1: (no value), rcl:P0817V
- added U$1: EI40-CUSTOM, untitled:EE40/EI40-DOWN
- added U$3: (no value), heatsink:SK104
- U$2: value TRANSFORMER-EE40-DOWN -> (none); device untitled:EE40/EI40-DOWN -> heatsink:SK104
- moved U$2 16.9 mm to (85.7, 47.9), turned to 180 degrees
Connections:
- new net GND: C2.2, IC1.7
- new net N$1: B1.AC2, U$1.P$14
- new net N$2: B1.AC1, U$1.P$8
- new net N$3: B1.-, C1.1, GND.B5
- new net N$4: C1.2, R1.1, VCC.B5
- new net N$5: B1.+, R1.2
- new net VCC: C2.1, IC1.12
Other:
- board size 100 x 70 mm -> 100 x 50 mm
Changed lines of the file:
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@@
 <setting verticaltext="up"/>
 </settings>
-<grid distance="10" unitdist="mm" unit="mm" style="lines" multiple="1" display="yes" altdistance="5" altunitdist="mil" altunit="mil"/>
+<grid distance="1" unitdist="mm" unit="mm" style="lines" multiple="1" display="yes" altdistance="5" altunitdist="mil" altunit="mil"/>
 <layers>
 <layer number="1" name="Top" color="4" fill="1" visible="yes" active="yes"/>
@@
 <plain>
 <wire x1="0" y1="0" x2="100" y2="0" width="0" layer="20"/>
-<wire x1="100" y1="0" x2="100" y2="70" width="0" layer="20"/>
-<wire x1="100" y1="70" x2="0" y2="70" width="0" layer="20"/>
-<wire x1="0" y1="70" x2="0" y2="40" width="0" layer="20"/>
-<wire x1="0" y1="40" x2="40" y2="40" width="0" layer="20"/>
-<wire x1="40" y1="40" x2="40" y2="30" width="0" layer="20"/>
-<wire x1="40" y1="30" x2="0" y2="30" width="0" layer="20"/>
-<wire x1="0" y1="30" x2="0" y2="0" width="0" layer="20"/>
+<wire x1="100" y1="0" x2="100" y2="50" width="0" layer="20"/>
+<wire x1="100" y1="50" x2="0" y2="50" width="0" layer="20"/>
+<wire x1="0" y1="50" x2="0" y2="0" width="0" layer="20"/>
+<circle x="15" y="25" radius="5" width="0.1524" layer="46"/>
 </plain>
 <attributes>
@@
 </autorouter>
 <elements>
-<element name="U$2" library="untitled" package="EE40/EI40-DOWN" value="TRANSFORMER-EE40-DOWN" x="73.208" y="36.477" smashed="yes"/>
+<element name="GND" library="holes" library_urn="urn:adsk.eagle:library:237" package="5,0-PAD-SQUARE" package3d_urn="urn:adsk.eagle:package:14298/1" value="MOUNT-PAD-SQUARE5.0" x="5.637" y="44.404" smashed="yes">
+<attribute name="POPULARITY" value="0" x="5.637" y="44.404" size="1.778" layer="27" display="off"/>
+</element>
+<element name="VCC" library="holes" library_urn="urn:adsk.eagle:library:237" package="5,0-PAD-SQUARE" package3d_urn="urn:adsk.eagle:package:14298/1" value="MOUNT-PAD-SQUARE5.0" x="5.541" y="5.541" smashed="yes">
+<attribute name="POPULARITY" value="0" x="5.541" y="5.541" size="1.778" layer="27" display="off"/>
+</element>
+<element name="B1" library="rectifier" library_urn="urn:adsk.eagle:library:336" package="GBU4S" package3d_urn="urn:adsk.eagle:package:23875/1" value="" x="23" y="37.016" smashed="yes" rot="R270">
+<attribute name="NAME" x="27.445" y="48.827" size="1.778" layer="25" ratio="10" rot="R270"/>
+<attribute name="POPULARITY" value="0" x="23" y="37.016" size="1.778" layer="27" rot="R270" display="off"/>
+<attribute name="VALUE" x="20.46" y="42.096" size="1.778" layer="27" ratio="10" rot="R270"/>
+</element>
+<element name="U$1" library="untitled" package="EE40/EI40-DOWN" value="EI40-CUSTOM" x="46.752" y="24.892" smashed="yes" rot="R180"/>
+<element name="U$2" library="heatsink" library_urn="urn:adsk.eagle:library:236" package="SK104" package3d_urn="urn:adsk.eagle:package:14176/1" value="" x="85.704" y="47.869" smashed="yes" rot="R180">
+<attribute name="VALUE" x="92.308" y="54.346" size="1.778" layer="27" ratio="10" rot="R180"/>
+</element>
+<element name="U$3" library="heatsink" library_urn="urn:adsk.eagle:library:236" package="SK104" package3d_urn="urn:adsk.eagle:package:14176/1" value="" x="85.831" y="2.35" smashed="yes">
+<attribute name="VALUE" x="79.227" y="-4.127" size="1.778" layer="27" ratio="10"/>
+</element>
+<element name="C1" library="capacitor-wima" library_urn="urn:adsk.eagle:library:116" package="C10B4" package3d_urn="urn:adsk.eagle:package:5400/1" value="" x="16.907" y="41.005" smashed="yes" rot="R270">
+<attribute name="NAME" x="19.32" y="44.434" size="1.27" layer="25" ratio="10" rot="R270"/>
+<attribute name="POPULARITY" value="0" x="16.907" y="41.005" size="1.778" layer="27" rot="R270" display="off"/>
+<attribute name="VALUE" x="15.256" y="42.529" size="1.27" layer="27" ratio="10" rot="R270"/>
+</element>
+<element name="R1" library="rcl" library_urn="urn:adsk.eagle:library:334" package="P0817V" package3d_urn="urn:adsk.eagle:package:23608/1" value="" x="17.911" y="11.876" smashed="yes" rot="R90">
+<attribute name="NAME" x="13.6946" y="3.494" size="1.27" layer="25" ratio="10" rot="R90"/>
+<attribute name="POPULARITY" value="0" x="17.911" y="11.876" size="1.778" layer="27" rot="R90" display="off"/>
+<attribute name="SPICEPREFIX" value="R" x="17.911" y="11.876" size="1.778" layer="27" rot="R90" display="off"/>
+<attribute name="VALUE" x="18.4952" y="5.653" size="1.27" layer="27" ratio="10" rot="R90"/>
+</element>
+<element name="Q1" library="transistor-power" library_urn="urn:adsk.eagle:library:400" package="TO220BV" package3d_urn="urn:adsk.eagle:package:29484/3" value="IRF740" x="85.826" y="2.446" smashed="yes" rot="R180">
+<attribute name="POPULARITY" value="0" x="85.826" y="2.446" size="1.778" layer="27" rot="R180" display="off"/>
+</element>
+<element name="Q2" library="transistor-power" library_urn="urn:adsk.eagle:library:400" package="TO220BV" package3d_urn="urn:adsk.eagle:package:29484/3" value="IRF740" x="85.664" y="47.815" smashed="yes">
+<attribute name="POPULARITY" value="0" x="85.664" y="47.815" size="1.778" layer="27" display="off"/>
+</element>
+<element name="IC1" library="linear" library_urn="urn:adsk.eagle:library:262" package="SO16" package3d_urn="urn:adsk.eagle:package:16423/2" value="TL494CD" x="77" y="35" smashed="yes">
+<attribute name="NAME" x="71.793" y="32.968" size="1.27" layer="25" ratio="10" rot="R90"/>
+<attribute name="POPULARITY" value="1" x="77" y="35" size="1.778" layer="27" display="off"/>
+<attribute name="VALUE" x="72.936" y="34.365" size="1.27" layer="27" ratio="10"/>
+</element>
+<element name="C2" library="capacitor-wima" library_urn="urn:adsk.eagle:library:116" package="C2.5-2" package3d_urn="urn:adsk.eagle:package:5415/1" value="" x="2" y="-9" smashed="yes">
+<attribute name="NAME" x="0.349" y="-7.476" size="1.27" layer="25" ratio="10"/>
+<attribute name="POPULARITY" value="28" x="2" y="-9" size="1.778" layer="27" display="off"/>
+<attribute name="VALUE" x="0.349" y="-11.794" size="1.27" layer="27" ratio="10"/>
+</element>
 </elements>
 <signals>
+<signal name="N$1">
+<contactref element="U$1" pad="P$14"/>
+<contactref element="B1" pad="AC2"/>
+<wire x1="23" y1="39.556" x2="34.12618125" y2="39.845475" width="0" layer="19" extent="1-1"/>
+</signal>
+<signal name="N$2">
+<contactref element="B1" pad="AC1"/>
+<contactref element="U$1" pad="P$8"/>
+<wire x1="34.12618125" y1="9.845475" x2="23" y2="34.476" width="0" layer="19" extent="1-1"/>
+</signal>
+<signal name="N$3">
+<contactref element="B1" pad="-"/>
+<contactref element="GND" pad="B5"/>
+<contactref element="C1" pad="1"/>
+<wire x1="23" y1="44.636" x2="5.637" y2="44.404" width="0" layer="19" extent="1-1"/>
+<wire x1="16.907" y1="46.085" x2="23" y2="44.636" width="0" layer="19" extent="1-1"/>
+</signal>
+<signal name="N$4">
+<contactref element="VCC" pad="B5"/>
+<contactref element="C1" pad="2"/>
+<contactref element="R1" pad="1"/>
+<wire x1="17.911" y1="6.796" x2="16.907" y2="35.925" width="0" layer="19" extent="1-1"/>
+<wire x1="5.541" y1="5.541" x2="17.911" y2="6.796" width="0" layer="19" extent="1-1"/>
+</signal>
+<signal name="N$5">
+<contactref element="B1" pad="+"/>
+<contactref element="R1" pad="2"/>
+<wire x1="17.911" y1="13.146" x2="23" y2="29.396" width="0" layer="19" extent="1-1"/>
+</signal>
+<signal name="GND">
+<contactref element="IC1" pad="7"/>
+<contactref element="C2" pad="2"/>
+<wire x1="3.27" y1="-9" x2="80.175" y2="31.9266" width="0" layer="19" extent="1-1"/>
+</signal>
+<signal name="VCC">
+<contactref element="IC1" pad="12"/>
+<contactref element="C2" pad="1"/>
+<wire x1="0.73" y1="-9" x2="77.635" y2="38.0734" width="0" layer="19" extent="1-1"/>
+</signal>
 </signals>
 <mfgpreviewcolors>
@@
 </board>
 </drawing>
+<compatibility>
+<note version="8.2" severity="warning">
+Since Version 8.2, EAGLE supports online libraries. The ids
+of those online libraries will not be understood (or retained)
+with this version.
+</note>
+<note version="8.3" severity="warning">
+Since Version 8.3, EAGLE supports URNs for individual library
+assets (packages, symbols, and devices). The URNs of those assets
+will not be understood (or retained) with this version.
+</note>
+<note version="8.3" severity="warning">
+Since Version 8.3, EAGLE supports the association of 3D packages
+with devices in libraries, schematics, and board files. Those 3D
+packages will not be understood (or retained) with this version.
+</note>
+</compatibility>
 </eagle>

Commit message: add
Parts:
- removed IC1: TL494CD, linear:SO16
- added D1, D2: 1N4148DO35-7, diode:DO35-7
- added D3, D4: 1N4148DO35-10, diode:DO35-10
- added R2, R3, R4, R5: (no value), rcl:0204/7
- added U$4: INDUCTOR-30A, untitled:INDUCTOR_30A
- C2: device capacitor-wima:C2.5-2 -> rcl:C225-062X268
- moved C2 74.5 mm to (68.4, 24.8), turned to 270 degrees
- moved B1 22.8 mm to (3.37, 25.4)
- moved C1 8.17 mm to (13.8, 33.4), turned to 0 degrees
- moved U$1 4.00 mm to (42.8, 24.9)
- moved Q1 0.37 mm to (85.8, 2.08)
- moved U$3 0.36 mm to (85.8, 1.99)
- moved Q2 0.05 mm to (85.6, 47.8)
- moved U$2 0.05 mm to (85.7, 47.9)
Connections:
- new net N$6: D1.C, D3.A, Q1.G, R2.2, R4.2
- new net N$7: D2.C, D4.A, Q2.G, R3.1, R5.2
- new net O1: C2.2, D4.C, Q1.D, U$1.P$1, U$1.P$2
- new net O2: C2.1, D3.C, Q2.D, U$1.P$6, U$1.P$7
- new net T4-2: U$1.P$3, U$1.P$4, U$1.P$5, U$4.P$1
- net GND: now also D1.A, D2.A, Q1.S, Q2.S, R2.1; no longer C2.2, IC1.7
- net VCC: now also R4.1, R5.1, U$4.P$2; no longer C2.1, IC1.12

Commit message: add
Parts:
- added GND2, VCC-BT: MOUNT-PAD-ROUND3.0, holes:3,0-PAD
- added LED1: TLLR4400, led:LED3MM
- added R6: 1m, rcl:0204/7
- C2: device rcl:C225-062X268 -> rcl:C225-108X268
- GND, VCC: value MOUNT-PAD-SQUARE5.0 -> MOUNT-PAD-ROUND3.0; device holes:5,0-PAD-SQUARE -> holes:3,0-PAD
- moved R4 31.2 mm to (68.5, 28.7), turned to 180 degrees
- moved D3 25.0 mm to (78.0, 29.6)
- moved Q2 16.1 mm to (73.8, 58.8)
- moved U$2 16.1 mm to (74.2, 59.2)
- moved D2 16.0 mm to (73.8, 51.5)
- moved R3 16.0 mm to (74.0, 49.1)
- moved C1 15.2 mm to (7.84, 47.4)
- moved R5 14.7 mm to (68.5, 31.1), flipped to the top, turned to 180 degrees
- moved R1 13.7 mm to (5.29, 17.3)
- moved Q1 12.8 mm to (73.0, 1.72)
- moved U$3 12.6 mm to (73.3, 0.88)
- moved GND 12.2 mm to (3.53, 56.4)
- moved R2 12.2 mm to (72.4, 10.9)
- moved D1 12.0 mm to (72.6, 8.34)
- moved D4 7.36 mm to (75.3, 29.6)
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Connections:
- removed net VCC: R4.1, R5.1, U$4.P$2
- new net N$8: R4.1, R5.1, U$4.P$2, VCC-BT.B3,0
- new net N$9: LED1.A, R6.2
- net GND: now also GND2.B3,0, R3.2
- net N$1: now also LED1.K
- net N$2: now also R6.1
- net N$3: now also GND.B3,0; no longer GND.B5
- net N$4: now also VCC.B3,0; no longer VCC.B5
Routing:
- net GND: track 0.00 -> 126.2 mm
- net N$4: track 0.00 -> 110.3 mm
- net T4-2: track 0.00 -> 90.9 mm
- net N$1: track 0.00 -> 83.9 mm
- net N$6: track 0.00 -> 61.0 mm
- net N$8: track 0.00 -> 59.7 mm, vias 0 -> 1
- net N$2: track 0.00 -> 54.9 mm
- net O2: track 0.00 -> 53.0 mm
- net N$7: track 0.00 -> 50.0 mm
- net O1: track 0.00 -> 49.0 mm
- net N$3: track 0.00 -> 17.0 mm
- net N$5: track 0.00 -> 6.98 mm
- net N$9: track 0.00 -> 2.80 mm
Other:
- board size 100 x 50 mm -> 100 x 60 mm
