File: untitled.brd (EAGLE design)
At the start: 100 x 60 mm, 12 parts

Commit message: add
Parts:
- added D2: 1N5060GP, diode:DO15-12
- added T1: E13005, transistor:TO220BV
- added U$10: (no value), heatsink:SK104
- added U$7, U$8: (no value), holes:3,0
- added U$9: IGBT-N-TO247, untitled:TO-247AD-V
- moved U$5 3.12 mm to (27.4, 57.3)
Connections:
- removed net N$2: R1.2, U$1.+, U$2.+, U$3.+, U$4.+
- new net IO: U$9.G
- net GND: now also R1.1, U$1.-, U$2.-, U$3.-, U$4.-, U$9.E
- net N$1: now also D2.C, T1.2; no longer R1.1, U$1.-, U$2.-, U$3.-, U$4.-
- net N$3: now also R1.2, T1.3, U$1.+, U$2.+, U$3.+, U$4.+
- net N$4: now also U$9.C
- net N$8: now also D2.A
Changed lines of the file:
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@@
 <setting verticaltext="up"/>
 </settings>
-<grid distance="15" unitdist="mm" unit="mm" style="lines" multiple="1" display="yes" altdistance="0.000123031496" altunitdist="mil" altunit="mil"/>
+<grid distance="0.625" unitdist="mm" unit="mm" style="lines" multiple="1" display="yes" altdistance="0.000123031496" altunitdist="mil" altunit="mil"/>
 <layers>
 <layer number="1" name="Top" color="4" fill="1" visible="yes" active="yes"/>
@@
 <attribute name="POPULARITY" value="17" x="95" y="5" size="1.778" layer="27" display="off"/>
 </element>
-<element name="U$5" library="heatsink" library_urn="urn:adsk.eagle:library:236" package="SK104" package3d_urn="urn:adsk.eagle:package:14176/1" value="" x="30.48" y="57.277" smashed="yes" rot="R180">
-<attribute name="NAME" x="37.084" y="61.595" size="1.778" layer="25" ratio="10" rot="R180"/>
-<attribute name="VALUE" x="37.084" y="63.754" size="1.778" layer="27" ratio="10" rot="R180"/>
+<element name="U$5" library="heatsink" library_urn="urn:adsk.eagle:library:236" package="SK104" package3d_urn="urn:adsk.eagle:package:14176/1" value="" x="27.355" y="57.277" smashed="yes" rot="R180">
+<attribute name="NAME" x="33.959" y="61.595" size="1.778" layer="25" ratio="10" rot="R180"/>
+<attribute name="VALUE" x="33.959" y="63.754" size="1.778" layer="27" ratio="10" rot="R180"/>
 </element>
 <element name="R1" library="rcl" library_urn="urn:adsk.eagle:library:334" package="0204/7" package3d_urn="urn:adsk.eagle:package:23498/2" value="" x="75" y="30" smashed="yes" rot="R180">
@@
 <attribute name="VALUE" x="7.989125" y="32.2725875" size="1.27" layer="28" ratio="10" rot="MR270"/>
 </element>
+<element name="U$7" library="holes" library_urn="urn:adsk.eagle:library:237" package="3,0" package3d_urn="urn:adsk.eagle:package:14277/1" value="" x="50" y="56.875" smashed="yes"/>
+<element name="U$8" library="holes" library_urn="urn:adsk.eagle:library:237" package="3,0" package3d_urn="urn:adsk.eagle:package:14277/1" value="" x="50" y="3.125" smashed="yes"/>
+<element name="U$9" library="untitled" package="TO-247AD-V" value="IGBT-N-TO247" x="27.27763125" y="56.943296875" smashed="yes">
+<attribute name="NAME" x="19.65763125" y="49.258296875" size="1.778" layer="25" ratio="10"/>
+<attribute name="VALUE" x="19.65763125" y="47.353296875" size="1.778" layer="27" ratio="10"/>
+</element>
+<element name="T1" library="transistor" library_urn="urn:adsk.eagle:library:402" package="TO220BV" package3d_urn="urn:adsk.eagle:package:28769/2" value="E13005" x="28.125" y="3.125" smashed="yes" rot="R180">
+<attribute name="NAME" x="33.205" y="9.1702" size="1.27" layer="25" ratio="10" rot="R180"/>
+<attribute name="POPULARITY" value="0" x="28.125" y="3.125" size="1.778" layer="27" rot="R180" display="off"/>
+<attribute name="VALUE" x="33.205" y="10.745" size="1.27" layer="27" ratio="10" rot="R180"/>
+</element>
+<element name="U$10" library="heatsink" library_urn="urn:adsk.eagle:library:236" package="SK104" package3d_urn="urn:adsk.eagle:package:14176/1" value="" x="27.645" y="2.723" smashed="yes">
+<attribute name="NAME" x="21.041" y="-1.595" size="1.778" layer="25" ratio="10"/>
+<attribute name="VALUE" x="21.041" y="-3.754" size="1.778" layer="27" ratio="10"/>
+</element>
+<element name="D2" library="diode" library_urn="urn:adsk.eagle:library:210" package="DO15-12" package3d_urn="urn:adsk.eagle:package:43369/2" value="1N5060GP" x="11.25" y="11.25" smashed="yes" rot="R180">
+<attribute name="NAME" x="14.933" y="9.091" size="1.27" layer="25" ratio="10" rot="R180"/>
+<attribute name="POPULARITY" value="0" x="11.25" y="11.25" size="1.778" layer="27" rot="R180" display="off"/>
+<attribute name="VALUE" x="13.409" y="12.647" size="1.27" layer="27" ratio="10" rot="R180"/>
+</element>
 </elements>
 <signals>
-<signal name="N$1">
+<signal name="GND">
+<contactref element="V-" pad="B3,0"/>
 <contactref element="U$1" pad="-"/>
 <contactref element="U$2" pad="-"/>
@@
 <contactref element="U$4" pad="-"/>
 <contactref element="R1" pad="1"/>
-<wire x1="68.779" y1="42.376" x2="91.24" y2="42.593" width="0" layer="19" extent="1-1"/>
-<wire x1="68.981" y1="17.202" x2="68.779" y2="42.376" width="0" layer="19" extent="1-1"/>
-<wire x1="91.277" y1="17.315" x2="68.981" y2="17.202" width="0" layer="19" extent="1-1"/>
-<wire x1="78.81" y1="30" x2="68.981" y2="17.202" width="0" layer="19" extent="1-1"/>
-</signal>
-<signal name="N$2">
+<contactref element="U$9" pad="E"/>
+<wire x1="78.81" y1="30" x2="91.24" y2="42.593" width="0" layer="19" extent="1-1"/>
+<wire x1="68.779" y1="42.376" x2="78.81" y2="30" width="0" layer="19" extent="1-1"/>
+<wire x1="68.981" y1="17.202" x2="78.81" y2="30" width="0" layer="19" extent="1-1"/>
+<wire x1="91.277" y1="17.315" x2="78.81" y2="30" width="0" layer="19" extent="1-1"/>
+<wire x1="32.77763125" y1="54.403296875" x2="68.779" y2="42.376" width="0" layer="19" extent="1-1"/>
+<wire x1="5" y1="55" x2="32.77763125" y2="54.403296875" width="0" layer="19" extent="1-1"/>
+</signal>
+<signal name="N$8">
+<contactref element="V+" pad="B3,0"/>
+<contactref element="D2" pad="A"/>
+<wire x1="4.9" y1="11.25" x2="5" y2="5" width="0" layer="19" extent="1-1"/>
+</signal>
+<signal name="N$3">
+<contactref element="D1" pad="C"/>
+<contactref element="U$6" pad="P$1"/>
 <contactref element="U$1" pad="+"/>
 <contactref element="U$2" pad="+"/>
@@
 <contactref element="U$4" pad="+"/>
 <contactref element="R1" pad="2"/>
-<wire x1="58.779" y1="42.376" x2="81.24" y2="42.593" width="0" layer="19" extent="1-1"/>
-<wire x1="58.981" y1="17.202" x2="58.779" y2="42.376" width="0" layer="19" extent="1-1"/>
-<wire x1="81.277" y1="17.315" x2="58.981" y2="17.202" width="0" layer="19" extent="1-1"/>
-<wire x1="71.19" y1="30" x2="58.981" y2="17.202" width="0" layer="19" extent="1-1"/>
-</signal>
-<signal name="GND">
-<contactref element="V-" pad="B3,0"/>
-</signal>
-<signal name="N$8">
-<contactref element="V+" pad="B3,0"/>
-</signal>
-<signal name="N$3">
-<contactref element="D1" pad="C"/>
-<contactref element="U$6" pad="P$1"/>
+<contactref element="T1" pad="3"/>
+<wire x1="71.19" y1="30" x2="81.24" y2="42.593" width="0" layer="19" extent="1-1"/>
+<wire x1="81.277" y1="17.315" x2="71.19" y2="30" width="0" layer="19" extent="1-1"/>
+<wire x1="58.779" y1="42.376" x2="71.19" y2="30" width="0" layer="19" extent="1-1"/>
+<wire x1="58.981" y1="17.202" x2="71.19" y2="30" width="0" layer="19" extent="1-1"/>
+<wire x1="25.585" y1="5.665" x2="58.981" y2="17.202" width="0" layer="19" extent="1-1"/>
+<wire x1="14.998715625" y1="40.00013125" x2="25.585" y2="5.665" width="0" layer="19" extent="1-1"/>
 <wire x1="5.830125" y1="37.3525875" x2="14.998715625" y2="40.00013125" width="0" layer="19" extent="1-1"/>
 </signal>
@@
 <contactref element="U$6" pad="P$2"/>
 <contactref element="D1" pad="A"/>
+<contactref element="U$9" pad="C"/>
+<wire x1="14.998715625" y1="20.00013125" x2="27.27763125" y2="54.403296875" width="0" layer="19" extent="1-1"/>
 <wire x1="5.830125" y1="22.1125875" x2="14.998715625" y2="20.00013125" width="0" layer="19" extent="1-1"/>
 </signal>
+<signal name="IO">
+<contactref element="U$9" pad="G"/>
+</signal>
+<signal name="N$1">
+<contactref element="D2" pad="C"/>
+<contactref element="T1" pad="2"/>
+<wire x1="17.6" y1="11.25" x2="28.125" y2="5.665" width="0" layer="19" extent="1-1"/>
+</signal>
 </signals>

Commit message: add
Parts:
- removed R1: (no value), rcl:0204/7
- added D4: (no value), zetex:E2LINE
- added OK1: SFH618A-3, optocoupler:DIP4
- added R2, R3: 10k, rcl:0207/2V
- added T2: 2N3565, transistor:TO92
- added U$11, U$12: RUBYCON_450V_270UF, untitled:RUBYCON_22*40
- moved U$3 5.93 mm to (64.7, 48.2), turned to 0 degrees
- turned U$1 to 0 degrees
- turned U$2 to 0 degrees
- turned U$4 to 0 degrees
- renumbered GND to BT-, VCC to BT+
Connections:
- net IO renamed SWITCH
- net N$8 renamed V+
- removed net GND: R1.1, U$1.-, U$2.-, U$3.-, U$4.-, U$9.E, V-.B3,0
- new net CHARGE: T1.1, T2.3
- new net N$2: D4.2, OK1.1
- new net N$5: OK1.3, R2.1, T2.2
- new net N$7: BT-.B3,0, OK1.4, T2.1
- new net V-: BT+.B3,0, OK1.2, R2.2, R3.1, U$1.-, U$2.-, U$3.-, U$4.-, U$9.E, V-.B3,0
- net N$3: now also D4.1, R3.2; no longer R1.2

Commit message: add
Parts:
- added LED1: TLLY4400, led:LED3MM
- added R1: 10k, rcl:0207/2V
- moved U$3 7.29 mm to (65.5, 41.0)
- moved U$2 2.40 mm to (88.1, 18.9)
- moved U$4 2.30 mm to (65.7, 18.7)
- moved U$1 2.01 mm to (87.7, 41.2)
- moved R3 1.83 mm to (77.4, 29.5)
- moved U$12 1.54 mm to (43.4, 19.2)
- moved U$5 0.91 mm to (28.2, 57.7)
- moved U$9 0.91 mm to (28.1, 57.3)
- moved U$11 0.45 mm to (43.3, 41.3)
- moved U$10 0.39 mm to (28.0, 2.61)
- moved T1 0.39 mm to (28.5, 3.01)
Connections:
- new net N$6: LED1.A, R1.2
- net CHARGE: now also R1.1
- net N$7: now also BT+.B3,0; no longer BT-.B3,0
- net V-: now also BT-.B3,0, LED1.K; no longer BT+.B3,0

Commit message: add
Parts:
- removed D4: (no value), zetex:E2LINE
- removed T1: E13005, transistor:TO220BV
- added D3, D5: (no value), zetex:E2LINE
- added Q1: FQPF10N60C, transistor-power:TO220BV
- added R4: 10k, rcl:0207/2V
- added R5: 100, rcl:0207/2V
- D2: value 1N5060GP -> FR307
- T2: value 2N3565 -> s8050
- moved OK1 5.00 mm to (78.1, 3.75)
- moved T2 2.50 mm to (61.3, 2.48)
- moved R2 2.23 mm to (77.8, 8.29)
- moved LED1 1.37 mm to (56.4, 2.35)
- turned U$6 to 180 degrees
- turned D1 to 90 degrees
Connections:
- removed net N$1: D2.C, T1.2
- new net N$10: D5.2, Q1.D, R3.1, U$1.-, U$11.-, U$12.-, U$2.-, U$3.-, U$4.-, U$9.E
- new net UC: D1.C, D2.C, D3.1, D5.1, R3.2, U$1.+, U$11.+, U$12.+, U$2.+, U$3.+, U$4.+, U$6.P$1
- net CHARGE: now also LED1.K, Q1.G, R4.2, T2.2; no longer R1.1, T1.1, T2.3
- net N$2: now also D3.2; no longer D4.2
- net N$3: now also R5.2, T2.1; no longer D1.C, D4.1, R3.2, T1.3, U$1.+, U$2.+, U$3.+, U$4.+, U$6.P$1
- net N$5: now also OK1.4, R5.1; no longer OK1.3, T2.2
- net N$7: now also OK1.3, R1.1, R4.1; no longer OK1.4, T2.1
- net V-: now also Q1.S, T2.3; no longer LED1.K, R3.1, U$1.-, U$2.-, U$3.-, U$4.-, U$9.E

Commit message: add
Parts:
- removed U$11, U$12: RUBYCON_450V_270UF, untitled:RUBYCON_22*40
- added U$13: IGBT-N-TO247, untitled:TO-247AD-V
- added U$14: (no value), heatsink:SK104
- D3: value (none) -> 400v
- moved D5 28.9 mm to (98.1, 30.1), turned to 180 degrees
- moved OK1 3.61 mm to (74.5, 3.35)
- moved D3 2.72 mm to (83.7, 2.58)
- moved R5 1.80 mm to (66.8, 1.94)
- moved R4 1.80 mm to (66.6, 5.85)
- moved LED1 1.04 mm to (56.6, 3.37)
- moved R2 0.55 mm to (77.3, 8.59)
Connections:
- net N$10: now also U$13.E; no longer U$11.-, U$12.-
- net N$4: now also U$13.C
- net UC: no longer U$11.+, U$12.+

Commit message: add
Parts:
- added D4: (no value), zetex:E2LINE
- added T1: S8050, transistor:TO92
- added X1: 22-23-2021, con-molex:22-23-2021
- moved T2 21.4 mm to (41.3, 10.1)
- moved R4 15.1 mm to (53.0, 12.5)
- moved R1 9.27 mm to (62.0, 2.42), turned to 180 degrees
- moved D5 2.07 mm to (96.0, 30.3)
- moved R2 2.03 mm to (75.6, 7.62)
- moved D3 1.46 mm to (82.4, 3.22), turned to 180 degrees
- moved LED1 0.39 mm to (56.7, 2.99), turned to 180 degrees
- moved R5 0.37 mm to (67.2, 2.10)
Connections:
- new net N$1: D4.2, T1.2
- net CHARGE: now also T1.1
- net SWITCH: now also U$13.G
- net UC: now also D4.1
- net V-: now also T1.3
Routing:
- net UC: track 0.00 -> 215.3 mm
- net N$10: track 0.00 -> 185.8 mm
- net V-: track 0.00 -> 160.4 mm, vias 0 -> 1
- net N$7: track 0.00 -> 106.2 mm
- net N$4: track 0.00 -> 103.7 mm
- net SWITCH: track 0.00 -> 53.0 mm
- net CHARGE: track 0.00 -> 38.0 mm
- net N$3: track 0.00 -> 29.9 mm
- net N$5: track 0.00 -> 9.91 mm
- net V+: track 0.00 -> 6.25 mm
- net N$2: track 0.00 -> 4.08 mm
- net N$1: track 0.00 -> 3.79 mm
- net N$6: track 0.00 -> 2.99 mm

Commit message: add
Parts:
- removed X1: 22-23-2021, con-molex:22-23-2021
- added J1: 61300311121, Headers:61300311121
Routing:
- net UC: track 215.3 -> 194.0 mm
- net CHARGE: track 38.0 -> 48.4 mm, vias 0 -> 1

Commit message: add
Parts:
- added OK2: SFH618A-3, optocoupler:DIP4
- added Q2: 2N3906, transistor-pnp:TO92
- added R10, R6, R7, R8, R9: 10k, rcl:0207/2V
- added T3: s8050, transistor:TO92
- moved J1 8.10 mm to (49.5, 41.0), turned to 180 degrees
Connections:
- removed net N$7: BT+.B3,0, OK1.3, R1.1, R4.1
- new net BT+: BT+.B3,0, OK1.4, OK2.4, R1.1, R4.1, R6.1
- new net N$11: J1.1, OK2.1
- new net N$12: OK2.3, Q2.2, R8.1, T3.1
- new net N$13: Q2.1, R7.1
- new net N$14: R6.2, T3.2
- new net N$8: Q2.3, R9.1, T3.3
- new net V2-: J1.2, OK2.2
- net N$10: now also R10.1
- net N$5: now also OK1.3; no longer OK1.4
- net SWITCH: now also R10.2, R9.2
- net V-: now also R7.2, R8.2
Routing:
- net BT+: track 0.00 -> 135.9 mm, vias 0 -> 1
- net N$7: track 106.2 -> 0.00 mm
- net V-: track 160.4 -> 188.8 mm
- net SWITCH: track 53.0 -> 78.8 mm
- net N$12: track 0.00 -> 15.6 mm
- net N$10: track 185.8 -> 195.7 mm
- net N$8: track 0.00 -> 8.80 mm
- net N$14: track 0.00 -> 7.00 mm
- net N$13: track 0.00 -> 6.27 mm
- net V2-: track 0.00 -> 2.82 mm
- net N$11: track 0.00 -> 2.82 mm
- net N$5: track 9.91 -> 8.54 mm
