File: untitled.brd (EAGLE design)
At the start: 100 x 60 mm, 40 parts, among them J1 61300311121, Q1 FQPF10N60C, Q2 2N3906, T1 S8050, T2 s8050, T3 s8050

Commit message: add
Parts:
- removed OK1: SFH618A-3, optocoupler:DIP4
- added D6, D7: (no value), zetex:E2LINE
- added Q3: s8550, transistor-pnp:TO92
- added R11: 10k, rcl:0207/2V
- Q2: value 2N3906 -> s8550
- R5: value 100 -> 2R
- moved R2 67.1 mm to (10.2, -7.62)
- moved R4 55.9 mm to (3.81, -14.0), turned to 0 degrees
- moved T2 51.6 mm to (3.81, -25.4)
- moved R5 28.4 mm to (76.7, 28.8)
- moved R3 20.3 mm to (57.1, 30.4), turned to 90 degrees
- moved D5 19.2 mm to (77.0, 33.1), turned to 90 degrees
Connections:
- net N$8 renamed STOPC
- removed net N$5: OK1.3, R2.1, R5.1
- removed net V2-: J1.2, OK2.2
- new net BT-: BT-.B3,0, J1.2, OK2.2, Q1.S, R11.2, R4.2, T1.3, V-.B3,0
- new net N$7: D3.2, Q3.2, R11.1, T2.1
- new net N$8: R4.1, T2.3
- new net N$9: Q3.3, R2.2
- net BT+: now also D7.1, J1.3, R2.1; no longer BT+.B3,0, OK1.4, R4.1
- net CHARGE: now also Q3.1; no longer R4.2
- net N$10: now also D6.2, R5.1; no longer D5.2
- net N$2: now also BT+.B3,0, D7.2; no longer D3.2, OK1.1
- net N$3: now also D5.2; no longer T2.1
- net N$4: now also D6.1
- net V-: no longer BT-.B3,0, OK1.2, Q1.S, R2.2, T1.3, T2.3, V-.B3,0
Routing:
- net V-: track 188.8 -> 84.8 mm
- net BT-: track 0.00 -> 81.5 mm
- net CHARGE: track 48.4 -> 7.27 mm, vias 1 -> 0
- net N$3: track 29.9 -> 0.00 mm
- net BT+: track 135.9 -> 117.2 mm
- net UC: track 194.0 -> 179.2 mm
- net STOPC: track 8.80 -> 20.8 mm, vias 0 -> 2
- net N$10: track 195.7 -> 187.1 mm
- net N$5: track 8.54 -> 0.00 mm
- net V2-: track 2.82 -> 0.00 mm
- net N$12: track 15.6 -> 12.9 mm
- net N$2: track 4.08 -> 5.71 mm

Commit message: add
Parts:
- removed D3: 400v, zetex:E2LINE
- removed D4: (no value), zetex:E2LINE
- removed T1: S8050, transistor:TO92
- added R12: 37k, rcl:0207/2V
- D5: value (none) -> 440v
- R3: value 10k -> 3k
- moved T2 50.6 mm to (35.6, 14.0), turned to 180 degrees
- moved Q3 49.6 mm to (35.6, 17.8)
- moved R4 45.5 mm to (40.6, 12.7), turned to 270 degrees
- moved R11 45.4 mm to (44.5, 12.7), turned to 270 degrees
- moved R2 32.5 mm to (30.5, 17.8), turned to 270 degrees
Connections:
- new net CVO: R12.1, R3.1
- net BT-: no longer T1.3
- net CHARGE: no longer T1.1
- net N$1: now also R11.1; no longer D4.2, T1.2
- net N$10: now also R3.2; no longer R3.1
- net N$7: no longer D3.2, R11.1
- net UC: now also R12.2; no longer D3.1, D4.1, R3.2
Routing:
- net N$10: track 187.1 -> 0.00 mm
- net UC: track 179.2 -> 0.00 mm
- net BT+: track 117.2 -> 0.00 mm, vias 1 -> 0
- net N$4: track 103.7 -> 0.00 mm
- net V-: track 84.8 -> 0.00 mm, vias 1 -> 0
- net BT-: track 81.5 -> 0.00 mm
- net SWITCH: track 78.8 -> 0.00 mm
- net STOPC: track 20.8 -> 0.00 mm, vias 2 -> 0
- net N$12: track 12.9 -> 0.00 mm
- net CHARGE: track 7.27 -> 0.00 mm
- net N$14: track 7.00 -> 0.00 mm
- net N$13: track 6.27 -> 0.00 mm
- net V+: track 6.25 -> 0.00 mm
- net N$2: track 5.71 -> 0.00 mm
- net N$1: track 3.79 -> 0.00 mm
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
Commit message: add
Parts:
- removed OK2: SFH618A-3, optocoupler:DIP4
- removed T2: s8050, transistor:TO92
- added IC1: LM393N, linear:DIL08
- added R13: 5.1k, rcl:0207/2V
- added R14: 2k, rcl:0207/2V
- added R15: 100k, rcl:0207/2V
- added R16: 1k, rcl:0207/2V
- added T1: s8050, transistor:TO92
- added VR1: (no value), v-reg:TO92-CLP
- R11: value 10k -> 470
- R12: value 37k -> 220k
- R3: value 3k -> 5.1k
- R5: value 2R -> 10R
- moved R3 27.5 mm to (73.9, 8.60), turned to 89.6 degrees
- moved R12 27.5 mm to (77.2, 11.0)
- moved R11 25.0 mm to (68.6, 6.35), turned to 0 degrees
- moved R4 14.3 mm to (26.7, 9.53), turned to 180 degrees
- moved R7 14.3 mm to (48.9, 23.4)
- moved R2 12.5 mm to (41.1, 11.2), turned to 180 degrees
- moved J1 9.74 mm to (50.8, 31.4), turned to 0 degrees
- moved T3 9.67 mm to (43.8, 22.5), turned to 89.5 degrees
- moved R9 9.00 mm to (43.9, 31.6), turned to 0 degrees
- moved Q2 8.81 mm to (43.6, 28.1), turned to 179.7 degrees
- moved R1 7.21 mm to (57.4, 8.00), turned to 270 degrees
- moved Q3 6.62 mm to (36.1, 11.2), turned to 270 degrees
- moved R8 5.57 mm to (49.1, 28.1), turned to 0 degrees
- moved R6 4.47 mm to (50.4, 25.7)
- moved LED1 0.85 mm to (55.9, 2.61)
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Connections:
- removed net N$14: R6.2, T3.2
- removed net N$9: Q3.3, R2.2
- removed net V-: R7.2, R8.2
- new net CIN: J1.1, Q2.2, R8.1, T3.1
- new net N$5: IC1.2, R11.2, R13.1, VR1.C
- net BT+: now also IC1.8, R11.1, R16.2; no longer OK2.4
- net BT-: now also IC1.4, R14.2, R7.2, R8.2, T1.1, VR1.A; no longer OK2.2, R11.2
- net CHARGE: now also R4.1, T1.3; no longer T2.2
- net CVO: now also IC1.3
- net N$1: now also IC1.1, Q3.2, R2.2; no longer R11.1
- net N$10: now also Q3.3, R16.1; no longer D6.2, Q1.D, R10.1, R3.2, R5.1, U$1.-, U$13.E, U$2.-, U$3.-, U$4.-, U$9.E
- net N$11: now also Q2.3, R6.2; no longer J1.1, OK2.1
- net N$12: now also Q2.1, R9.1, T3.2; no longer OK2.3, Q2.2, R8.1, T3.1
- net N$13: now also T3.3; no longer Q2.1
- net N$7: now also R13.2, R14.1, VR1.R; no longer Q3.2, T2.1
- net N$8: now also D6.2, Q1.D, R10.1, R15.2, R3.2, R5.1, U$1.-, U$13.E, U$2.-, U$3.-, U$4.-, U$9.E; no longer R4.1, T2.3
- net STOPC: now also T1.2; no longer Q2.3, R9.1, T3.3
- net UC: now also R15.1
Routing:
- net BT-: track 0.00 -> 157.1 mm
- net BT+: track 0.00 -> 105.2 mm
- net N$8: track 0.00 -> 84.2 mm
- net UC: track 0.00 -> 43.6 mm
- net CHARGE: track 0.00 -> 33.2 mm
- net N$4: track 0.00 -> 13.3 mm
- net N$1: track 0.00 -> 9.22 mm
- net V+: track 0.00 -> 6.55 mm
- net N$2: track 0.00 -> 6.01 mm
- net N$10: track 0.00 -> 4.52 mm
- net N$3: track 0.00 -> 4.41 mm
- net N$6: track 0.00 -> 4.20 mm
- net CVO: track 0.00 -> 4.15 mm
- net N$7: track 0.00 -> 2.54 mm

Commit message: add
Parts:
- removed T1: s8050, transistor:TO92
- added Q4: s8550, transistor-pnp:TO92
Connections:
- removed net STOPC: T1.2
- net BT-: now also Q4.1; no longer T1.1
- net CHARGE: now also Q4.3; no longer T1.3
- net CIN: now also Q4.2
Routing:
- net N$8: track 84.2 -> 29.6 mm
- net BT-: track 157.1 -> 122.2 mm
- net CHARGE: track 33.2 -> 19.7 mm
Changed lines of the file:
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@@
 <attribute name="SPICEPREFIX" value="R" x="41.275" y="13.843" size="1.778" layer="27" display="off"/>
-</element>
-<element name="T1" library="transistor" library_urn="urn:adsk.eagle:library:402" package="TO92" package3d_urn="urn:adsk.eagle:package:28523/2" value="s8050" x="32.004" y="11.176" smashed="yes" rot="R90">
-<attribute name="NAME" x="31.369" y="14.351" size="1.27" layer="25" ratio="10" rot="R90"/>
-<attribute name="POPULARITY" value="0" x="32.004" y="11.176" size="1.778" layer="27" rot="R90" display="off"/>
-<attribute name="VALUE" x="33.274" y="14.351" size="1.27" layer="27" ratio="10" rot="R90"/>
 </element>
 <element name="R8" library="rcl" library_urn="urn:adsk.eagle:library:334" package="0207/2V" package3d_urn="urn:adsk.eagle:package:23490/1" value="10k" x="49.149" y="28.067" smashed="yes">
@@
 <attribute name="POPULARITY" value="17" x="49.149" y="28.067" size="1.778" layer="27" display="off"/>
 <attribute name="SPICEPREFIX" value="R" x="49.149" y="28.067" size="1.778" layer="27" display="off"/>
+</element>
+<element name="Q4" library="transistor-pnp" library_urn="urn:adsk.eagle:library:399" package="TO92" package3d_urn="urn:adsk.eagle:package:29211/2" value="s8550" x="31.242" y="10.414" smashed="yes" rot="R270">
+<attribute name="NAME" x="31.877" y="7.239" size="1.27" layer="25" ratio="10" rot="R270"/>
+<attribute name="POPULARITY" value="11" x="31.242" y="10.414" size="1.778" layer="27" rot="R270" display="off"/>
+<attribute name="VALUE" x="29.972" y="7.239" size="1.27" layer="27" ratio="10" rot="R270"/>
 </element>
 </elements>
@@
 <contactref element="Q3" pad="1"/>
 <contactref element="R4" pad="1"/>
-<contactref element="T1" pad="3"/>
-<wire x1="27.94" y1="9.525" x2="31.623" y2="9.525" width="1.016" layer="16"/>
-<wire x1="30.861" y1="5.467696875" x2="30.7393375" y2="5.346034375" width="1.016" layer="16"/>
-<wire x1="31.623" y1="9.525" x2="32.004" y2="9.906" width="1.016" layer="16" curve="90"/>
-<wire x1="32.004" y1="9.906" x2="32.004" y2="6.610696875" width="1.016" layer="16"/>
-<wire x1="32.004" y1="6.610696875" x2="30.7393375" y2="5.346034375" width="1.016" layer="16" curve="-90"/>
-<wire x1="36.068" y1="9.906" x2="32.004" y2="9.906" width="1.016" layer="16"/>
 <wire x1="36.068" y1="9.906" x2="36.068" y2="9.144" width="1.016" layer="16"/>
 <wire x1="36.068" y1="9.144" x2="38.608" y2="6.604" width="1.016" layer="16" curve="90"/>
 <wire x1="54.644896875" y1="3.683" x2="54.644896875" y2="2.611459375" width="1.016" layer="16"/>
 <wire x1="38.608" y1="6.604" x2="52.866896875" y2="6.604" width="1.016" layer="16"/>
+<contactref element="Q4" pad="3"/>
 <wire x1="52.866896875" y1="6.604" x2="54.644896875" y2="3.683" width="0" layer="19" extent="16-16"/>
+<wire x1="31.242" y1="11.684" x2="36.068" y2="9.906" width="0" layer="19" extent="1-1"/>
+<wire x1="27.94" y1="9.525" x2="31.242" y2="11.684" width="0" layer="19" extent="1-1"/>
+<wire x1="30.7393375" y1="5.346034375" x2="27.94" y2="9.525" width="0" layer="19" extent="1-1"/>
 </signal>
 <signal name="N$6">
@@
 <wire x1="57.399021875" y1="6.7271" x2="57.184896875" y2="6.512975" width="1.016" layer="16"/>
 <wire x1="57.184896875" y1="2.611459375" x2="57.184896875" y2="6.512975" width="1.016" layer="16"/>
-</signal>
-<signal name="STOPC">
-<contactref element="T1" pad="2"/>
 </signal>
 <signal name="UC">
@@
 <contactref element="T3" pad="1"/>
 <contactref element="R8" pad="1"/>
-<wire x1="43.551025" y1="26.162025" x2="48.26" y2="31.369" width="0" layer="19" extent="1-1"/>
+<contactref element="Q4" pad="2"/>
+<wire x1="47.879" y1="28.067" x2="48.26" y2="31.369" width="0" layer="19" extent="1-1"/>
+<wire x1="43.551025" y1="26.162025" x2="47.879" y2="28.067" width="0" layer="19" extent="1-1"/>
 <wire x1="43.82608125" y1="23.74895" x2="43.551025" y2="26.162025" width="0" layer="19" extent="1-1"/>
-<wire x1="47.879" y1="28.067" x2="43.82608125" y2="23.74895" width="0" layer="19" extent="1-1"/>
+<wire x1="33.147" y1="10.414" x2="43.82608125" y2="23.74895" width="0" layer="19" extent="1-1"/>
 </signal>
 <signal name="BT-">
@@
 <contactref element="VR1" pad="A"/>
 <contactref element="R14" pad="2"/>
-<contactref element="T1" pad="1"/>
-<wire x1="25.6593375" y1="5.346034375" x2="25.6593375" y2="9.2656625" width="1.016" layer="16"/>
 <wire x1="25.6593375" y1="9.2656625" x2="25.4" y2="9.525" width="1.016" layer="16"/>
-<wire x1="32.004" y1="12.446" x2="31.75" y2="12.7" width="1.016" layer="16" curve="90"/>
-<wire x1="31.75" y1="12.7" x2="28.1993375" y2="12.7" width="1.016" layer="16"/>
-<wire x1="28.1993375" y1="12.7" x2="25.6593375" y2="10.16" width="1.016" layer="16" curve="90"/>
-<wire x1="25.6593375" y1="10.16" x2="25.6593375" y2="9.2656625" width="1.016" layer="16"/>
 <wire x1="25.4" y1="9.525" x2="24.765" y2="8.89" width="1.016" layer="16" curve="-90"/>
 <wire x1="24.765" y1="8.89" x2="11.43" y2="8.89" width="1.016" layer="16"/>
@@
 <wire x1="2.54" y1="17.78" x2="2.54" y2="52.54" width="1.016" layer="16"/>
 <wire x1="53.721" y1="8.89" x2="51.562" y2="6.731" width="1.016" layer="1" curve="-90"/>
-<wire x1="36.576" y1="6.731" x2="34.036" y2="9.271" width="1.016" layer="1" curve="-90"/>
-<wire x1="34.036" y1="10.414" x2="32.004" y2="12.446" width="1.016" layer="1" curve="90"/>
-<wire x1="51.562" y1="6.731" x2="36.576" y2="6.731" width="1.016" layer="1"/>
-<wire x1="34.036" y1="9.271" x2="34.036" y2="10.414" width="1.016" layer="1"/>
 <wire x1="77.343" y1="3.81" x2="78.498765625" y2="3.81" width="1.27" layer="16"/>
 <wire x1="78.498765625" y1="3.81" x2="80.645" y2="4.699" width="1.27" layer="16" curve="45"/>
@@
 <contactref element="R7" pad="2"/>
 <contactref element="R8" pad="2"/>
-<wire x1="50.165" y1="23.368" x2="50.8" y2="31.369" width="0" layer="19" extent="1-1"/>
-<wire x1="50.419" y1="28.067" x2="50.165" y2="23.368" width="0" layer="19" extent="1-1"/>
-<wire x1="32.004" y1="12.446" x2="50.419" y2="28.067" width="0" layer="19" extent="1-1"/>
+<contactref element="Q4" pad="1"/>
+<wire x1="50.419" y1="28.067" x2="50.8" y2="31.369" width="0" layer="19" extent="1-1"/>
+<wire x1="50.165" y1="23.368" x2="50.419" y2="28.067" width="0" layer="19" extent="1-1"/>
+<wire x1="53.721" y1="8.89" x2="50.165" y2="23.368" width="0" layer="19" extent="1-1"/>
+<wire x1="31.242" y1="9.144" x2="51.562" y2="6.731" width="0" layer="19" extent="1-1"/>
+<wire x1="25.6593375" y1="9.2656625" x2="31.242" y2="9.144" width="0" layer="19" extent="16-16"/>
+<wire x1="25.6593375" y1="5.346034375" x2="25.6593375" y2="9.2656625" width="0" layer="19" extent="16-16"/>
 </signal>
 <signal name="N$2">
@@
 <contactref element="R5" pad="1"/>
 <contactref element="R3" pad="2"/>
-<wire x1="28.1993375" y1="5.346034375" x2="28.1993375" y2="4.826" width="1.27" layer="1"/>
-<wire x1="28.1993375" y1="4.826" x2="25.6593375" y2="2.286" width="1.27" layer="1" curve="-90"/>
-<wire x1="25.273" y1="2.286" x2="22.733" y2="4.826" width="1.27" layer="1" curve="-90"/>
-<wire x1="22.733" y1="9.398" x2="25.273" y2="11.938" width="1.27" layer="1" curve="-90"/>
-<wire x1="27.432" y1="11.938" x2="28.575" y2="13.081" width="1.27" layer="1" curve="90"/>
-<wire x1="28.575" y1="13.081" x2="30.734" y2="15.24" width="1.27" layer="1" curve="-90"/>
-<wire x1="37.846" y1="15.24" x2="38.608" y2="16.002" width="1.27" layer="1" curve="90"/>
-<wire x1="38.608" y1="16.002" x2="38.608" y2="16.1617125" width="1.27" layer="1"/>
-<wire x1="38.608" y1="16.1617125" x2="41.148" y2="18.7017125" width="1.27" layer="1" curve="-90"/>
-<wire x1="41.148" y1="18.7017125" x2="60.722659375" y2="18.7017125" width="1.27" layer="1"/>
-<wire x1="25.6593375" y1="2.286" x2="25.273" y2="2.286" width="1.27" layer="1"/>
-<wire x1="22.733" y1="4.826" x2="22.733" y2="9.398" width="1.27" layer="1"/>
-<wire x1="25.273" y1="11.938" x2="27.432" y2="11.938" width="1.27" layer="1"/>
-<wire x1="30.734" y1="15.24" x2="37.846" y2="15.24" width="1.27" layer="1"/>
 <wire x1="73.877915625" y1="9.86951875" x2="73.877915625" y2="10.15998125" width="1.27" layer="1"/>
 <wire x1="77.978" y1="28.829" x2="90.57095" y2="28.829" width="1.27" layer="1"/>
@@
 <wire x1="24.384" y1="48.641" x2="33.59901875" y2="54.802040625" width="0" layer="19" extent="1-1"/>
 <wire x1="17.272" y1="50.419" x2="24.384" y2="48.641" width="0" layer="19" extent="1-1"/>
+<wire x1="28.1993375" y1="5.346034375" x2="60.722659375" y2="18.7017125" width="0" layer="19" extent="1-1"/>
 </signal>
 <signal name="N$10">
@@
 <wire x1="44.83098125" y1="28.06035" x2="49.149" y2="25.654" width="0" layer="19" extent="1-1"/>
 </signal>
-<signal name="N$12">
-<contactref element="Q2" pad="1"/>
-<contactref element="T3" pad="2"/>
-<contactref element="R9" pad="1"/>
-<wire x1="42.291015625" y1="28.073646875" x2="42.672" y2="31.623" width="0" layer="19" extent="1-1"/>
-<wire x1="41.910071875" y1="22.495621875" x2="42.291015625" y2="28.073646875" width="0" layer="19" extent="1-1"/>
-</signal>
 <signal name="N$13">
 <contactref element="T3" pad="3"/>
@@
 <wire x1="43.803915625" y1="21.209046875" x2="47.625" y2="23.368" width="0" layer="19" extent="1-1"/>
 </signal>
+<signal name="N$9">
+<contactref element="R9" pad="1"/>
+<contactref element="Q2" pad="1"/>
+<contactref element="T3" pad="2"/>
+<wire x1="42.291015625" y1="28.073646875" x2="42.672" y2="31.623" width="0" layer="19" extent="1-1"/>
+<wire x1="41.910071875" y1="22.495621875" x2="42.291015625" y2="28.073646875" width="0" layer="19" extent="1-1"/>
+</signal>
 </signals>

Commit message: add
Parts:
- added OK1: SFH618A-4, optocoupler:DIP4
- added R17: 10k, rcl:0207/2V
- R6: value 10k -> 100k
- R9: device rcl:0207/2V -> rcl:0309/12
- moved D6 22.4 mm to (39.6, 50.9), turned to 270 degrees
- moved R9 16.2 mm to (30.4, 40.4), turned to 121.5 degrees
- moved VR1 11.0 mm to (69.8, 4.57), turned to 90 degrees
- moved T3 10.1 mm to (34.9, 17.8)
- moved R8 9.58 mm to (41.7, 22.1)
- moved R7 9.58 mm to (41.4, 17.4)
- moved J1 9.58 mm to (43.3, 25.4)
- moved R6 9.58 mm to (42.9, 19.7)
- moved Q2 9.44 mm to (35.3, 23.5)
- moved R14 5.57 mm to (72.9, 8.38), turned to 180 degrees
- moved R11 4.07 mm to (66.0, 3.17), turned to 90 degrees
- moved R1 3.95 mm to (59.6, 4.70)
- moved R3 3.89 mm to (76.9, 11.0)
- moved R12 3.32 mm to (79.6, 8.76)
- moved R13 3.32 mm to (74.3, 4.19), turned to 270 degrees
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Connections:
- new net N$12: OK1.1, R17.1
- new net N$14: OK1.3, Q2.2, R8.1, T3.1
- net BT+: no longer R6.1
- net BT-: now also OK1.2; no longer R7.2, R8.2
- net CIN: now also R17.2; no longer Q2.2, R8.1, T3.1
- net N$11: now also OK1.4
- net N$4: now also R6.1
- net N$8: now also R7.2, R8.2
Routing:
- net N$8: track 29.6 -> 311.8 mm
- net UC: track 43.6 -> 175.7 mm
- net N$4: track 13.3 -> 142.0 mm, vias 0 -> 1
- net BT-: track 122.2 -> 217.3 mm
- net SWITCH: track 0.00 -> 74.6 mm
- net N$5: track 0.22 -> 35.5 mm
- net CVO: track 4.15 -> 31.0 mm
- net CIN: track 0.00 -> 24.9 mm
- net N$9: track 0.00 -> 22.5 mm
- net CHARGE: track 19.7 -> 36.9 mm
- net BT+: track 105.2 -> 120.0 mm
- net N$14: track 0.00 -> 12.6 mm
- net N$11: track 0.00 -> 11.5 mm
- net N$7: track 2.54 -> 11.7 mm
- net N$1: track 9.22 -> 15.4 mm
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
Commit message: add
Parts:
- added R18: 10k, rcl:0207/2V
- R6: value 100k -> 200k
- R7, R8: value 10k -> 20k
- R9: value 10k -> 1k
Connections:
- net N$11: now also R18.1
- net N$8: now also R18.2
Routing:
- net N$11: track 11.5 -> 22.7 mm
- net N$8: track 311.8 -> 315.8 mm
Changed lines of the file:
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@@
 <attribute name="POPULARITY" value="11" x="35.306" y="23.495" size="1.778" layer="27" rot="R179.7" display="off"/>
 </element>
-<element name="R6" library="rcl" library_urn="urn:adsk.eagle:library:334" package="0207/2V" package3d_urn="urn:adsk.eagle:package:23490/1" value="100k" x="42.926" y="19.685" smashed="yes" rot="R180">
+<element name="R6" library="rcl" library_urn="urn:adsk.eagle:library:334" package="0207/2V" package3d_urn="urn:adsk.eagle:package:23490/1" value="200k" x="42.926" y="19.685" smashed="yes" rot="R180">
 <attribute name="NAME" x="47.6758" y="20.066" size="1.27" layer="25" ratio="10" rot="R180"/>
 <attribute name="POPULARITY" value="17" x="42.926" y="19.685" size="1.778" layer="27" rot="R180" display="off"/>
 <attribute name="SPICEPREFIX" value="R" x="42.926" y="19.685" size="1.778" layer="27" rot="R180" display="off"/>
 </element>
-<element name="R7" library="rcl" library_urn="urn:adsk.eagle:library:334" package="0207/2V" package3d_urn="urn:adsk.eagle:package:23490/1" value="10k" x="41.402" y="17.399" smashed="yes">
+<element name="R7" library="rcl" library_urn="urn:adsk.eagle:library:334" package="0207/2V" package3d_urn="urn:adsk.eagle:package:23490/1" value="20k" x="41.402" y="17.399" smashed="yes">
 <attribute name="NAME" x="43.5102" y="17.145" size="1.27" layer="25" ratio="10"/>
 <attribute name="POPULARITY" value="17" x="41.402" y="17.399" size="1.778" layer="27" display="off"/>
 <attribute name="SPICEPREFIX" value="R" x="41.402" y="17.399" size="1.778" layer="27" display="off"/>
 </element>
-<element name="R9" library="rcl" library_urn="urn:adsk.eagle:library:334" package="0309/12" package3d_urn="urn:adsk.eagle:package:23571/1" value="10k" x="30.353" y="40.386" smashed="yes" rot="R121.5">
+<element name="R9" library="rcl" library_urn="urn:adsk.eagle:library:334" package="0309/12" package3d_urn="urn:adsk.eagle:package:23571/1" value="1k" x="30.353" y="40.386" smashed="yes" rot="R121.5">
 <attribute name="NAME" x="29.513259375" y="39.811825" size="1.27" layer="25" ratio="10" rot="R121.5"/>
 <attribute name="POPULARITY" value="6" x="30.353" y="40.386" size="1.778" layer="27" rot="R121.5" display="off"/>
@@
 <attribute name="SPICEPREFIX" value="R" x="41.275" y="13.843" size="1.778" layer="27" display="off"/>
 </element>
-<element name="R8" library="rcl" library_urn="urn:adsk.eagle:library:334" package="0207/2V" package3d_urn="urn:adsk.eagle:package:23490/1" value="10k" x="41.656" y="22.098" smashed="yes">
+<element name="R8" library="rcl" library_urn="urn:adsk.eagle:library:334" package="0207/2V" package3d_urn="urn:adsk.eagle:package:23490/1" value="20k" x="41.656" y="22.098" smashed="yes">
 <attribute name="NAME" x="43.8912" y="21.59" size="1.27" layer="25" ratio="10"/>
 <attribute name="POPULARITY" value="17" x="41.656" y="22.098" size="1.778" layer="27" display="off"/>
@@
 <attribute name="POPULARITY" value="17" x="40.513" y="32.512" size="1.778" layer="27" rot="R270" display="off"/>
 <attribute name="SPICEPREFIX" value="R" x="40.513" y="32.512" size="1.778" layer="27" rot="R270" display="off"/>
+</element>
+<element name="R18" library="rcl" library_urn="urn:adsk.eagle:library:334" package="0207/2V" package3d_urn="urn:adsk.eagle:package:23490/1" value="10k" x="50.8" y="24.13" smashed="yes">
+<attribute name="NAME" x="50.7492" y="25.146" size="1.27" layer="25" ratio="10"/>
+<attribute name="POPULARITY" value="17" x="50.8" y="24.13" size="1.778" layer="27" display="off"/>
+<attribute name="SPICEPREFIX" value="R" x="50.8" y="24.13" size="1.778" layer="27" display="off"/>
+<attribute name="VALUE" x="50.7492" y="21.8948" size="1.27" layer="27" ratio="10"/>
 </element>
 </elements>
@@
 <wire x1="43.942" y1="17.399" x2="42.672" y2="17.399" width="0.4064" layer="1"/>
 <wire x1="51.308" y1="18.669" x2="45.212" y2="18.669" width="0.4064" layer="1"/>
+<contactref element="R18" pad="2"/>
+<wire x1="52.07" y1="24.13" x2="52.07" y2="20.828" width="0.4064" layer="1"/>
+<wire x1="52.07" y1="20.828" x2="52.578" y2="20.32" width="0.4064" layer="1" curve="90"/>
 </signal>
 <signal name="N$10">
@@
 <wire x1="37.973" y1="26.162" x2="36.57598125" y2="24.76498125" width="0.508" layer="16" curve="90"/>
 <wire x1="36.57598125" y1="24.76498125" x2="36.57598125" y2="23.48835" width="0.508" layer="16"/>
+<contactref element="R18" pad="1"/>
+<wire x1="49.53" y1="24.13" x2="48.768" y2="23.368" width="0.4064" layer="1" curve="-90"/>
+<wire x1="48.768" y1="23.368" x2="42.672" y2="23.368" width="0.4064" layer="1"/>
+<wire x1="42.672" y1="23.368" x2="41.656" y2="22.352" width="0.4064" layer="1" curve="90"/>
+<wire x1="41.656" y1="22.352" x2="41.656" y2="19.685" width="0.4064" layer="1"/>
 </signal>
 <signal name="N$13">
