File: untitled.sch (EAGLE design)
At the start: 1 part

Commit message: add
Parts:
- removed U$1: TRANSFORMER-EE40, untitled:TRANSFORMER-EE40
- added U$2: TRANSFORMER-EE40-DOWN, untitled:TRANSFORMER-EE40-DOWN
Changed lines of the file:
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@@
 </classes>
 <parts>
-<part name="U$1" library="untitled" deviceset="TRANSFORMER-EE40" device=""/>
+<part name="U$2" library="untitled" deviceset="TRANSFORMER-EE40-DOWN" device=""/>
 </parts>
 <sheets>
@@
 </plain>
 <instances>
-<instance part="U$1" gate="G$1" x="35.56" y="33.02" smashed="yes">
-<attribute name="NAME" x="31.75" y="45.72" size="1.778" layer="95"/>
+<instance part="U$2" gate="G$1" x="68.58" y="30.48" smashed="yes">
+<attribute name="NAME" x="64.77" y="48.26" size="1.778" layer="95"/>
 </instance>
 </instances>

Commit message: add
Parts:
- removed U$2: TRANSFORMER-EE40-DOWN, untitled:TRANSFORMER-EE40-DOWN
- added B1: (no value), rectifier:GBU4S
- added C1: (no value), capacitor-wima:C10/4
- added C2: (no value), capacitor-wima:C2.5/2
- added GND, VCC: MOUNT-PAD-SQUARE5.0, holes:MOUNT-PAD-SQUARE5.0
- added IC1: TL494CD, linear:TL494CD
- added Q1, Q2: IRF740, transistor-power:IRF740
- added R1: (no value), rcl:R-US_0817/7V
- added U$1: EI40-CUSTOM, untitled:EI40-CUSTOM
Connections:
- new net GND: C2.2
- new net N$1: B1.AC1, U$1.T4-2
- new net N$2: B1.AC2, U$1.T4-1
- new net N$3: B1.-, C1.1, GND.MOUNT
- new net N$4: C1.2, R1.1, VCC.MOUNT
- new net N$5: B1.+, R1.2
- new net VCC: C2.1

Commit message: add
Parts:
- removed IC1: TL494CD, linear:TL494CD
- added D1, D2: 1N4148DO35-7, diode:1N4148DO35-7
- added D3, D4: 1N4148DO35-10, diode:1N4148DO35-10
- added R2, R3, R4, R5: (no value), rcl:R-EU_0204/7
- added U$4: INDUCTOR-30A, untitled:INDUCTOR-30A
- C2: device capacitor-wima:C2.5/2 -> rcl:C-EU225-062X268
Connections:
- new net N$6: D1.C, D3.A, Q1.G, R2.2, R4.2
- new net N$7: D2.C, D4.A, Q2.G, R3.1, R5.2
- new net O1: C2.2, D4.C, Q1.D, U$1.T1
- new net O2: C2.1, D3.C, Q2.D, U$1.T3
- new net T4-2: U$1.T2, U$4.1
- net GND: now also D1.A, D2.A, Q1.S, Q2.S, R2.1; no longer C2.2
- net VCC: now also R4.1, R5.1, U$4.2; no longer C2.1
Other:
- moved on the sheet: C2, Q1, Q2

Commit message: add
Parts:
- added GND2, VCC-BT: MOUNT-PAD-ROUND3.0, holes:MOUNT-PAD-ROUND3.0
- added LED1: TLLR4400, led:TLLR4400
- added R6: 1m, rcl:R-EU_0204/7
- C2: device rcl:C-EU225-062X268 -> rcl:C-EU225-108X268
- GND, VCC: value MOUNT-PAD-SQUARE5.0 -> MOUNT-PAD-ROUND3.0; device holes:MOUNT-PAD-SQUARE5.0 -> holes:MOUNT-PAD-ROUND3.0
Connections:
- removed net VCC: R4.1, R5.1, U$4.2
- new net N$8: R4.1, R5.1, U$4.2, VCC-BT.MOUNT
- new net N$9: LED1.A, R6.2
- net GND: now also GND2.MOUNT, R3.2
- net N$1: now also LED1.C
- net N$2: now also R6.1
Changed lines of the file:
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@@
 </layers>
 <schematic xreflabel="%F%N/%S.%C%R" xrefpart="/%S.%C%R">
+<fusionteam huburn="a.YnVzaW5lc3M6Z21haWwxMjM3MjQz" projecturn="a.YnVzaW5lc3M6Z21haWwxMjM3MjQzI0QyMDIwMTAxODM0NDEzMjIwNg" folderUrn="urn:adsk.wipprod:fs.folder:co.L-SEJ-iYQoS1nu5sfy5KIw" urn="urn:adsk.wipprod:dm.lineage:OiMYtNLNTQa0Mq7WxEbOTw"  versionUrn="urn:adsk.wipprod:fs.file:vf.OiMYtNLNTQa0Mq7WxEbOTw?version=1" camFileUrn="" camFileVersionUrn="" lastpublishedchangeguid="032816dd-5246-b3cd-18d3-979e08d4332c"/>
 <attributes>
 </attributes>
@@
 </classes>
 <parts>
-<part name="GND" library="holes" library_urn="urn:adsk.eagle:library:237" deviceset="MOUNT-PAD-SQUARE" device="5.0" package3d_urn="urn:adsk.eagle:package:14298/1"/>
-<part name="VCC" library="holes" library_urn="urn:adsk.eagle:library:237" deviceset="MOUNT-PAD-SQUARE" device="5.0" package3d_urn="urn:adsk.eagle:package:14298/1"/>
+<part name="GND" library="holes" library_urn="urn:adsk.eagle:library:237" deviceset="MOUNT-PAD-ROUND" device="3.0" package3d_urn="urn:adsk.eagle:package:14280/1" value="MOUNT-PAD-ROUND3.0"/>
+<part name="VCC" library="holes" library_urn="urn:adsk.eagle:library:237" deviceset="MOUNT-PAD-ROUND" device="3.0" package3d_urn="urn:adsk.eagle:package:14280/1" value="MOUNT-PAD-ROUND3.0"/>
 <part name="B1" library="rectifier" library_urn="urn:adsk.eagle:library:336" deviceset="GBU4S" device="" package3d_urn="urn:adsk.eagle:package:23875/1"/>
 <part name="U$1" library="untitled" deviceset="EI40-CUSTOM" device=""/>
@@
 <part name="Q1" library="transistor-power" library_urn="urn:adsk.eagle:library:400" deviceset="IRF740" device="" package3d_urn="urn:adsk.eagle:package:29484/3"/>
 <part name="Q2" library="transistor-power" library_urn="urn:adsk.eagle:library:400" deviceset="IRF740" device="" package3d_urn="urn:adsk.eagle:package:29484/3"/>
-<part name="SUPPLY1" library="supply2" library_urn="urn:adsk.eagle:library:372" deviceset="VCC" device=""/>
 <part name="U$4" library="untitled" deviceset="INDUCTOR-30A" device=""/>
 <part name="SUPPLY2" library="supply2" library_urn="urn:adsk.eagle:library:372" deviceset="GND" device=""/>
@@
 <part name="R2" library="rcl" library_urn="urn:adsk.eagle:library:334" deviceset="R-EU_" device="0204/7" package3d_urn="urn:adsk.eagle:package:23498/2"/>
 <part name="R3" library="rcl" library_urn="urn:adsk.eagle:library:334" deviceset="R-EU_" device="0204/7" package3d_urn="urn:adsk.eagle:package:23498/2"/>
-<part name="C2" library="rcl" library_urn="urn:adsk.eagle:library:334" deviceset="C-EU" device="225-062X268" package3d_urn="urn:adsk.eagle:package:23661/1"/>
+<part name="C2" library="rcl" library_urn="urn:adsk.eagle:library:334" deviceset="C-EU" device="225-108X268" package3d_urn="urn:adsk.eagle:package:23663/1"/>
 <part name="R4" library="rcl" library_urn="urn:adsk.eagle:library:334" deviceset="R-EU_" device="0204/7" package3d_urn="urn:adsk.eagle:package:23498/2"/>
 <part name="R5" library="rcl" library_urn="urn:adsk.eagle:library:334" deviceset="R-EU_" device="0204/7" package3d_urn="urn:adsk.eagle:package:23498/2"/>
 <part name="D3" library="diode" library_urn="urn:adsk.eagle:library:210" deviceset="1N4148" device="DO35-10" package3d_urn="urn:adsk.eagle:package:43344/2"/>
 <part name="D4" library="diode" library_urn="urn:adsk.eagle:library:210" deviceset="1N4148" device="DO35-10" package3d_urn="urn:adsk.eagle:package:43344/2"/>
+<part name="VCC-BT" library="holes" library_urn="urn:adsk.eagle:library:237" deviceset="MOUNT-PAD-ROUND" device="3.0" package3d_urn="urn:adsk.eagle:package:14280/1" value="MOUNT-PAD-ROUND3.0"/>
+<part name="GND2" library="holes" library_urn="urn:adsk.eagle:library:237" deviceset="MOUNT-PAD-ROUND" device="3.0" package3d_urn="urn:adsk.eagle:package:14280/1" value="MOUNT-PAD-ROUND3.0"/>
+<part name="SUPPLY1" library="supply2" library_urn="urn:adsk.eagle:library:372" deviceset="GND" device=""/>
+<part name="LED1" library="led" library_urn="urn:adsk.eagle:library:259" deviceset="TLLR4400" device="" package3d_urn="urn:adsk.eagle:package:15797/1"/>
+<part name="R6" library="rcl" library_urn="urn:adsk.eagle:library:334" deviceset="R-EU_" device="0204/7" package3d_urn="urn:adsk.eagle:package:23498/2" value="1m"/>
 </parts>
 <sheets>
@@
 <attribute name="NAME" x="105.41" y="83.82" size="1.778" layer="95" rot="MR180"/>
 </instance>
-<instance part="SUPPLY1" gate="G$1" x="12.7" y="134.62" smashed="yes" rot="R90">
-<attribute name="VALUE" x="9.525" y="132.715" size="1.778" layer="96" rot="R90"/>
-</instance>
 <instance part="U$4" gate="G$1" x="55.88" y="134.62" smashed="yes" rot="R270">
 <attribute name="NAME" x="62.23" y="132.08" size="1.778" layer="95" rot="R270"/>
@@
 <instance part="D4" gate="G$1" x="106.68" y="96.52" smashed="yes" rot="R90">
 <attribute name="NAME" x="106.1974" y="99.06" size="1.778" layer="95" rot="R90"/>
+</instance>
+<instance part="VCC-BT" gate="G$1" x="12.7" y="134.62" smashed="yes" rot="R180">
+<attribute name="NAME" x="9.906" y="134.0358" size="1.778" layer="95" rot="R180"/>
+<attribute name="VALUE" x="9.906" y="137.0838" size="1.778" layer="96" rot="R180"/>
+</instance>
+<instance part="GND2" gate="G$1" x="15.24" y="91.44" smashed="yes" rot="R180">
+<attribute name="NAME" x="12.446" y="90.8558" size="1.778" layer="95" rot="R180"/>
+<attribute name="VALUE" x="12.446" y="93.9038" size="1.778" layer="96" rot="R180"/>
+</instance>
+<instance part="SUPPLY1" gate="GND" x="30.48" y="91.44" smashed="yes" rot="R90">
+<attribute name="VALUE" x="33.655" y="89.535" size="1.778" layer="96" rot="R90"/>
+</instance>
+<instance part="LED1" gate="G$1" x="83.82" y="38.1" smashed="yes" rot="R180">
+<attribute name="NAME" x="80.264" y="42.672" size="1.778" layer="95" rot="R270"/>
+</instance>
+<instance part="R6" gate="G$1" x="83.82" y="25.4" smashed="yes" rot="R90">
+<attribute name="NAME" x="82.3214" y="21.59" size="1.778" layer="95" rot="R90"/>
+<attribute name="VALUE" x="87.122" y="21.59" size="1.778" layer="96" rot="R90"/>
 </instance>
 </instances>
@@
 <pinref part="U$1" gate="G$1" pin="T4-2"/>
 <pinref part="B1" gate="1" pin="AC1"/>
-<wire x1="86.36" y1="45.72" x2="73.66" y2="45.72" width="0.1524" layer="91"/>
+<wire x1="86.36" y1="45.72" x2="83.82" y2="45.72" width="0.1524" layer="91"/>
+<wire x1="83.82" y1="45.72" x2="73.66" y2="45.72" width="0.1524" layer="91"/>
 <wire x1="73.66" y1="45.72" x2="73.66" y2="33.02" width="0.1524" layer="91"/>
+<pinref part="LED1" gate="G$1" pin="C"/>
+<wire x1="83.82" y1="45.72" x2="83.82" y2="43.18" width="0.1524" layer="91"/>
+<junction x="83.82" y="45.72"/>
 </segment>
 </net>
@@
 <pinref part="U$1" gate="G$1" pin="T4-1"/>
 <wire x1="73.66" y1="22.86" x2="73.66" y2="12.7" width="0.1524" layer="91"/>
-<wire x1="73.66" y1="12.7" x2="86.36" y2="12.7" width="0.1524" layer="91"/>
+<wire x1="73.66" y1="12.7" x2="83.82" y2="12.7" width="0.1524" layer="91"/>
+<pinref part="R6" gate="G$1" pin="1"/>
+<wire x1="83.82" y1="12.7" x2="86.36" y2="12.7" width="0.1524" layer="91"/>
+<wire x1="83.82" y1="20.32" x2="83.82" y2="12.7" width="0.1524" layer="91"/>
+<junction x="83.82" y="12.7"/>
 </segment>
 </net>
@@
 <pinref part="R1" gate="G$1" pin="2"/>
 <wire x1="66.04" y1="10.16" x2="78.74" y2="10.16" width="0.1524" layer="91"/>
-</segment>
-</net>
-<net name="VCC" class="0">
-<segment>
-<pinref part="SUPPLY1" gate="G$1" pin="VCC"/>
-<wire x1="15.24" y1="134.62" x2="43.18" y2="134.62" width="0.1524" layer="91"/>
-<pinref part="U$4" gate="G$1" pin="2"/>
-<pinref part="R4" gate="G$1" pin="1"/>
-<pinref part="R5" gate="G$1" pin="1"/>
-<wire x1="43.18" y1="134.62" x2="48.26" y2="134.62" width="0.1524" layer="91"/>
-<wire x1="76.2" y1="119.38" x2="76.2" y2="88.9" width="0.1524" layer="91"/>
-<wire x1="76.2" y1="119.38" x2="43.18" y2="119.38" width="0.1524" layer="91"/>
-<wire x1="43.18" y1="119.38" x2="43.18" y2="134.62" width="0.1524" layer="91"/>
-<junction x="76.2" y="119.38"/>
-<junction x="43.18" y="134.62"/>
 </segment>
 </net>
@@
 <wire x1="119.38" y1="106.68" x2="119.38" y2="91.44" width="0.1524" layer="91"/>
 <junction x="119.38" y="106.68"/>
+<pinref part="R3" gate="G$1" pin="2"/>
+<wire x1="96.52" y1="104.14" x2="96.52" y2="106.68" width="0.1524" layer="91"/>
+</segment>
+<segment>
+<pinref part="GND2" gate="G$1" pin="MOUNT"/>
+<pinref part="SUPPLY1" gate="GND" pin="GND"/>
+<wire x1="17.78" y1="91.44" x2="27.94" y2="91.44" width="0.1524" layer="91"/>
 </segment>
 </net>
@@
 </segment>
 </net>
+<net name="N$8" class="0">
+<segment>
+<wire x1="15.24" y1="134.62" x2="43.18" y2="134.62" width="0.1524" layer="91"/>
+<pinref part="U$4" gate="G$1" pin="2"/>
+<pinref part="R4" gate="G$1" pin="1"/>
+<pinref part="R5" gate="G$1" pin="1"/>
+<wire x1="43.18" y1="134.62" x2="48.26" y2="134.62" width="0.1524" layer="91"/>
+<wire x1="76.2" y1="119.38" x2="76.2" y2="88.9" width="0.1524" layer="91"/>
+<wire x1="76.2" y1="119.38" x2="43.18" y2="119.38" width="0.1524" layer="91"/>
+<wire x1="43.18" y1="119.38" x2="43.18" y2="134.62" width="0.1524" layer="91"/>
+<junction x="76.2" y="119.38"/>
+<junction x="43.18" y="134.62"/>
+<pinref part="VCC-BT" gate="G$1" pin="MOUNT"/>
+</segment>
+</net>
+<net name="N$9" class="0">
+<segment>
+<pinref part="LED1" gate="G$1" pin="A"/>
+<pinref part="R6" gate="G$1" pin="2"/>
+<wire x1="83.82" y1="35.56" x2="83.82" y2="30.48" width="0.1524" layer="91"/>
+</segment>
+</net>
