File: untitled.sch (EAGLE design)
At the start: 11 parts

Commit message: add
Parts:
- added D2: 1N5060GP, diode:1N5060GP
- added T1: E13005, transistor:2SC1306
- added U$9: IGBT-N-TO247, untitled:IGBT-N-TO247
Connections:
- removed net N$2: R1.2, U$1.+, U$2.+, U$3.+, U$4.+
- new net IO: U$9.G
- net GND: now also R1.1, U$1.-, U$2.-, U$3.-, U$4.-, U$9.E
- net N$1: now also D2.C, T1.C; no longer R1.1, U$1.-, U$2.-, U$3.-, U$4.-
- net N$3: now also R1.2, T1.E, U$1.+, U$2.+, U$3.+, U$4.+
- net N$4: now also U$9.C
- net N$8: now also D2.A
Other:
- moved on the sheet: R1, V+, V-

Commit message: add
Parts:
- removed GND, VCC: MOUNT-PAD-ROUND3.0, holes:MOUNT-PAD-ROUND3.0
- removed R1: (no value), rcl:R-US_0204/7
- added BT+, BT-: MOUNT-PAD-ROUND3.0, holes:MOUNT-PAD-ROUND3.0
- added D4: (no value), zetex:DS_E2L
- added OK1: SFH618A-3, optocoupler:SFH618A-3
- added R2, R3: 10k, rcl:R-EU_0207/2V
- added T2: 2N3565, transistor:2N3565
- added U$11, U$12: RUBYCON_450V_270UF, untitled:RUBYCON_450V_270UF
Connections:
- net IO renamed SWITCH
- net N$8 renamed V+
- removed net GND: R1.1, U$1.-, U$2.-, U$3.-, U$4.-, U$9.E, V-.MOUNT
- new net CHARGE: T1.B, T2.E
- new net N$2: D4.A, OK1.A
- new net N$5: OK1.EMIT, R2.1, T2.B
- new net N$7: BT-.MOUNT, OK1.COL, T2.C
- new net V-: BT+.MOUNT, OK1.C, R2.2, R3.1, U$1.-, U$2.-, U$3.-, U$4.-, U$9.E, V-.MOUNT
- net N$3: now also D4.K, R3.2; no longer R1.2

Commit message: add
Parts:
- added LED1: TLLY4400, led:TLLY4400
- added R1: 10k, rcl:R-EU_0207/2V
Connections:
- new net N$6: LED1.A, R1.2
- net CHARGE: now also R1.1
- net N$7: now also BT+.MOUNT; no longer BT-.MOUNT
- net V-: now also BT-.MOUNT, LED1.C; no longer BT+.MOUNT
Other:
- moved on the sheet: BT+, BT-, V-
Changed lines of the file:
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@@
 <part name="U$11" library="untitled" deviceset="RUBYCON_450V_270UF" device=""/>
 <part name="U$12" library="untitled" deviceset="RUBYCON_450V_270UF" device=""/>
+<part name="LED1" library="led" library_urn="urn:adsk.eagle:library:259" deviceset="TLLY4400" device="" package3d_urn="urn:adsk.eagle:package:15797/1"/>
+<part name="R1" library="rcl" library_urn="urn:adsk.eagle:library:334" deviceset="R-EU_" device="0207/2V" package3d_urn="urn:adsk.eagle:package:23490/1" value="10k"/>
 </parts>
 <sheets>
@@
 <attribute name="VALUE" x="-10.414" y="55.8038" size="1.778" layer="96" rot="R180"/>
 </instance>
-<instance part="V-" gate="G$1" x="-7.62" y="17.78" smashed="yes" rot="R180">
-<attribute name="NAME" x="-10.414" y="17.1958" size="1.778" layer="95" rot="R180"/>
-<attribute name="VALUE" x="-10.414" y="20.2438" size="1.778" layer="96" rot="R180"/>
-</instance>
-<instance part="BT+" gate="G$1" x="124.46" y="40.64" smashed="yes">
-<attribute name="NAME" x="127.254" y="41.2242" size="1.778" layer="95"/>
-<attribute name="VALUE" x="127.254" y="38.1762" size="1.778" layer="96"/>
-</instance>
-<instance part="BT-" gate="G$1" x="124.46" y="55.88" smashed="yes">
-<attribute name="NAME" x="127.254" y="56.4642" size="1.778" layer="95"/>
-<attribute name="VALUE" x="127.254" y="53.4162" size="1.778" layer="96"/>
+<instance part="V-" gate="G$1" x="-7.62" y="10.16" smashed="yes" rot="R180">
+<attribute name="NAME" x="-10.414" y="9.5758" size="1.778" layer="95" rot="R180"/>
+<attribute name="VALUE" x="-10.414" y="12.6238" size="1.778" layer="96" rot="R180"/>
+</instance>
+<instance part="BT+" gate="G$1" x="132.08" y="63.5" smashed="yes">
+<attribute name="NAME" x="134.874" y="64.0842" size="1.778" layer="95"/>
+<attribute name="VALUE" x="134.874" y="61.0362" size="1.778" layer="96"/>
+</instance>
+<instance part="BT-" gate="G$1" x="132.08" y="40.64" smashed="yes">
+<attribute name="NAME" x="134.874" y="41.2242" size="1.778" layer="95"/>
+<attribute name="VALUE" x="134.874" y="38.1762" size="1.778" layer="96"/>
 </instance>
 <instance part="U$6" gate="G$1" x="83.82" y="25.4" smashed="yes" rot="R270"/>
@@
 </instance>
 <instance part="T2" gate="G$1" x="99.06" y="50.8" smashed="yes">
-<attribute name="NAME" x="104.14" y="48.26" size="1.778" layer="95"/>
-<attribute name="VALUE" x="101.6" y="50.8" size="1.778" layer="96"/>
+<attribute name="NAME" x="93.98" y="50.8" size="1.778" layer="95"/>
+<attribute name="VALUE" x="91.44" y="53.34" size="1.778" layer="96"/>
 </instance>
 <instance part="R3" gate="G$1" x="63.5" y="24.638" smashed="yes" rot="R90">
@@
 <attribute name="VALUE" x="66.802" y="20.828" size="1.778" layer="96" rot="R90"/>
 </instance>
-<instance part="U$11" gate="G$1" x="0" y="30.988" smashed="yes"/>
-<instance part="U$12" gate="G$1" x="5.08" y="30.988" smashed="yes"/>
+<instance part="U$11" gate="G$1" x="0" y="25.908" smashed="yes"/>
+<instance part="U$12" gate="G$1" x="7.62" y="25.908" smashed="yes"/>
+<instance part="LED1" gate="G$1" x="119.38" y="45.72" smashed="yes"/>
+<instance part="R1" gate="G$1" x="111.76" y="55.88" smashed="yes">
+<attribute name="NAME" x="107.95" y="57.3786" size="1.778" layer="95"/>
+<attribute name="VALUE" x="107.95" y="52.578" size="1.778" layer="96"/>
+</instance>
 </instances>
 <busses>
@@
 <wire x1="78.74" y1="5.08" x2="40.64" y2="5.08" width="0.1524" layer="91"/>
 <wire x1="40.64" y1="5.08" x2="40.64" y2="18.796" width="0.1524" layer="91"/>
-<wire x1="-5.08" y1="17.78" x2="5.08" y2="17.78" width="0.1524" layer="91"/>
-<wire x1="5.08" y1="17.78" x2="27.94" y2="17.78" width="0.1524" layer="91"/>
-<wire x1="27.94" y1="17.78" x2="27.94" y2="18.796" width="0.1524" layer="91"/>
-<label x="7.62" y="15.24" size="1.778" layer="95"/>
+<wire x1="-5.08" y1="10.16" x2="5.08" y2="10.16" width="0.1524" layer="91"/>
+<wire x1="5.08" y1="10.16" x2="27.94" y2="10.16" width="0.1524" layer="91"/>
+<wire x1="27.94" y1="10.16" x2="27.94" y2="18.796" width="0.1524" layer="91"/>
+<label x="7.62" y="7.62" size="1.778" layer="95"/>
 <pinref part="R3" gate="G$1" pin="1"/>
 <pinref part="R2" gate="G$1" pin="2"/>
-<pinref part="BT+" gate="G$1" pin="MOUNT"/>
 <wire x1="114.3" y1="40.64" x2="119.38" y2="40.64" width="0.1524" layer="91"/>
-<wire x1="119.38" y1="40.64" x2="121.92" y2="40.64" width="0.1524" layer="91"/>
 <wire x1="119.38" y1="40.64" x2="119.38" y2="0" width="0.1524" layer="91"/>
 <wire x1="119.38" y1="0" x2="5.08" y2="0" width="0.1524" layer="91"/>
 <junction x="119.38" y="40.64"/>
-<wire x1="5.08" y1="0" x2="5.08" y2="17.78" width="0.1524" layer="91"/>
-<junction x="5.08" y="17.78"/>
+<wire x1="5.08" y1="0" x2="5.08" y2="10.16" width="0.1524" layer="91"/>
+<junction x="5.08" y="10.16"/>
+<pinref part="LED1" gate="G$1" pin="C"/>
+<pinref part="BT-" gate="G$1" pin="MOUNT"/>
+<wire x1="119.38" y1="40.64" x2="129.54" y2="40.64" width="0.1524" layer="91"/>
 </segment>
 <segment>
@@
 <segment>
 <pinref part="OK1" gate="G$1" pin="COL"/>
-<pinref part="BT-" gate="G$1" pin="MOUNT"/>
-<wire x1="88.9" y1="45.72" x2="88.9" y2="55.88" width="0.1524" layer="91"/>
-<wire x1="88.9" y1="55.88" x2="101.6" y2="55.88" width="0.1524" layer="91"/>
+<wire x1="88.9" y1="45.72" x2="88.9" y2="63.5" width="0.1524" layer="91"/>
+<pinref part="BT+" gate="G$1" pin="MOUNT"/>
+<wire x1="88.9" y1="63.5" x2="101.6" y2="63.5" width="0.1524" layer="91"/>
 <pinref part="T2" gate="G$1" pin="C"/>
-<wire x1="101.6" y1="55.88" x2="121.92" y2="55.88" width="0.1524" layer="91"/>
-<junction x="101.6" y="55.88"/>
+<wire x1="101.6" y1="63.5" x2="129.54" y2="63.5" width="0.1524" layer="91"/>
+<wire x1="101.6" y1="63.5" x2="101.6" y2="55.88" width="0.1524" layer="91"/>
+<junction x="101.6" y="63.5"/>
 </segment>
 </net>
@@
 <segment>
 <pinref part="T2" gate="G$1" pin="E"/>
-<wire x1="101.6" y1="45.72" x2="114.3" y2="45.72" width="0.1524" layer="91"/>
-<label x="109.22" y="45.72" size="1.778" layer="95"/>
+<wire x1="101.6" y1="45.72" x2="106.68" y2="45.72" width="0.1524" layer="91"/>
+<label x="104.14" y="45.72" size="1.778" layer="95"/>
+<pinref part="R1" gate="G$1" pin="1"/>
+<wire x1="106.68" y1="45.72" x2="114.3" y2="45.72" width="0.1524" layer="91"/>
+<wire x1="106.68" y1="55.88" x2="106.68" y2="45.72" width="0.1524" layer="91"/>
+<junction x="106.68" y="45.72"/>
 </segment>
 <segment>
@@
 </segment>
 </net>
+<net name="N$6" class="0">
+<segment>
+<pinref part="R1" gate="G$1" pin="2"/>
+<pinref part="LED1" gate="G$1" pin="A"/>
+<wire x1="116.84" y1="55.88" x2="119.38" y2="55.88" width="0.1524" layer="91"/>
+<wire x1="119.38" y1="55.88" x2="119.38" y2="48.26" width="0.1524" layer="91"/>
+</segment>
+</net>
+<net name="N$8" class="0">
+<segment>
+<junction x="101.6" y="63.5"/>
+</segment>
+</net>

Commit message: add
Parts:
- removed D4: (no value), zetex:DS_E2L
- removed T1: E13005, transistor:2SC1306
- added D3, D5: (no value), zetex:DS_E2L
- added Q1: FQPF10N60C, transistor-power:IRF740
- added R4: 10k, rcl:R-EU_0207/2V
- added R5: 100, rcl:R-EU_0207/2V
- D2: value 1N5060GP -> FR307
- T2: value 2N3565 -> s8050; device transistor:2N3565 -> transistor:2N3704
Connections:
- removed net N$1: D2.C, T1.C
- new net N$10: D5.A, Q1.D, R3.1, U$1.-, U$11.-, U$12.-, U$2.-, U$3.-, U$4.-, U$9.E
- new net UC: D1.C, D2.C, D3.K, D5.K, R3.2, U$1.+, U$11.+, U$12.+, U$2.+, U$3.+, U$4.+, U$6.1
- net CHARGE: now also LED1.C, Q1.G, R4.2, T2.C; no longer R1.1, T1.B, T2.E
- net N$2: now also D3.A; no longer D4.A
- net N$3: now also R5.2, T2.B; no longer D1.C, D4.K, R3.2, T1.E, U$1.+, U$2.+, U$3.+, U$4.+, U$6.1
- net N$5: now also OK1.COL, R5.1; no longer OK1.EMIT, T2.B
- net N$7: now also OK1.EMIT, R1.1, R4.1; no longer OK1.COL, T2.C
- net V-: now also Q1.S, T2.E; no longer LED1.C, R3.1, U$1.-, U$2.-, U$3.-, U$4.-, U$9.E
Other:
- moved on the sheet: BT+, BT-, D2, OK1, R1, R2, V+, V-

Commit message: add
Parts:
- removed U$11, U$12: RUBYCON_450V_270UF, untitled:RUBYCON_450V_270UF
- added U$13: IGBT-N-TO247, untitled:IGBT-N-TO247
- D3: value (none) -> 400v
Connections:
- net N$10: now also U$13.E; no longer U$11.-, U$12.-
- net N$4: now also U$13.C
- net UC: no longer U$11.+, U$12.+
Changed lines of the file:
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@@
 <part name="R2" library="rcl" library_urn="urn:adsk.eagle:library:334" deviceset="R-EU_" device="0207/2V" package3d_urn="urn:adsk.eagle:package:23490/1" value="10k"/>
 <part name="R3" library="rcl" library_urn="urn:adsk.eagle:library:334" deviceset="R-EU_" device="0207/2V" package3d_urn="urn:adsk.eagle:package:23490/1" value="10k"/>
-<part name="U$11" library="untitled" deviceset="RUBYCON_450V_270UF" device=""/>
-<part name="U$12" library="untitled" deviceset="RUBYCON_450V_270UF" device=""/>
 <part name="LED1" library="led" library_urn="urn:adsk.eagle:library:259" deviceset="TLLY4400" device="" package3d_urn="urn:adsk.eagle:package:15797/1"/>
 <part name="R1" library="rcl" library_urn="urn:adsk.eagle:library:334" deviceset="R-EU_" device="0207/2V" package3d_urn="urn:adsk.eagle:package:23490/1" value="10k"/>
@@
 <part name="Q1" library="transistor-power" library_urn="urn:adsk.eagle:library:400" deviceset="IRF740" device="" package3d_urn="urn:adsk.eagle:package:29484/3" value="FQPF10N60C"/>
 <part name="D5" library="zetex" deviceset="DS_E2L" device="" package3d_urn="urn:adsk.eagle:package:30989/1"/>
-<part name="D3" library="zetex" deviceset="DS_E2L" device="" package3d_urn="urn:adsk.eagle:package:30989/1"/>
+<part name="D3" library="zetex" deviceset="DS_E2L" device="" package3d_urn="urn:adsk.eagle:package:30989/1" value="400v"/>
+<part name="U$13" library="untitled" deviceset="IGBT-N-TO247" device=""/>
 </parts>
 <sheets>
@@
 <attribute name="VALUE" x="66.802" y="20.828" size="1.778" layer="96" rot="R90"/>
 </instance>
-<instance part="U$11" gate="G$1" x="-5.08" y="25.908" smashed="yes"/>
-<instance part="U$12" gate="G$1" x="5.08" y="25.908" smashed="yes"/>
 <instance part="LED1" gate="G$1" x="86.36" y="83.82" smashed="yes"/>
 <instance part="R1" gate="G$1" x="86.36" y="91.44" smashed="yes" rot="R270">
@@
 <attribute name="NAME" x="2.54" y="67.945" size="1.778" layer="95" rot="R180"/>
 <attribute name="VALUE" x="2.54" y="70.485" size="1.778" layer="96" rot="R180"/>
+</instance>
+<instance part="U$13" gate="G$1" x="86.36" y="12.7" smashed="yes">
+<attribute name="VALUE" x="89.916" y="13.081" size="1.778" layer="96"/>
 </instance>
 </instances>
@@
 <pinref part="U$9" gate="G$1" pin="C"/>
 <junction x="78.74" y="17.78"/>
+<pinref part="U$13" gate="G$1" pin="C"/>
+<wire x1="83.82" y1="17.78" x2="88.9" y2="17.78" width="0.1524" layer="91"/>
+<junction x="83.82" y="17.78"/>
 </segment>
 </net>
@@
 <junction x="5.08" y="5.08"/>
 <pinref part="Q1" gate="G$1" pin="S"/>
-</segment>
-<segment>
-<pinref part="OK1" gate="G$1" pin="C"/>
-<wire x1="20.32" y1="63.5" x2="7.62" y2="63.5" width="0.1524" layer="91"/>
-<label x="7.62" y="63.5" size="1.778" layer="95"/>
 </segment>
 <segment>
@@
 <label x="86.36" y="60.96" size="1.778" layer="95"/>
 </segment>
+<segment>
+<wire x1="20.32" y1="63.5" x2="-12.7" y2="63.5" width="0.1524" layer="91"/>
+<label x="-12.7" y="63.5" size="1.778" layer="95"/>
+<pinref part="OK1" gate="G$1" pin="C"/>
+</segment>
 </net>
 <net name="N$5" class="0">
@@
 <net name="N$10" class="0">
 <segment>
-<pinref part="U$11" gate="G$1" pin="-"/>
-<pinref part="U$12" gate="G$1" pin="-"/>
-<wire x1="-5.08" y1="18.796" x2="5.08" y2="18.796" width="0.1524" layer="91"/>
+<wire x1="-12.7" y1="18.796" x2="15.24" y2="18.796" width="0.1524" layer="91"/>
 <pinref part="U$4" gate="G$1" pin="-"/>
 <pinref part="R3" gate="G$1" pin="1"/>
@@
 <wire x1="15.24" y1="18.796" x2="27.94" y2="18.796" width="0.1524" layer="91"/>
 <wire x1="27.94" y1="15.24" x2="27.94" y2="18.796" width="0.1524" layer="91"/>
-<wire x1="5.08" y1="18.796" x2="15.24" y2="18.796" width="0.1524" layer="91"/>
-<junction x="5.08" y="18.796"/>
 <junction x="15.24" y="18.796"/>
 <pinref part="Q1" gate="G$1" pin="D"/>
 <wire x1="-12.7" y1="22.86" x2="-12.7" y2="18.796" width="0.1524" layer="91"/>
-<wire x1="-12.7" y1="18.796" x2="-5.08" y2="18.796" width="0.1524" layer="91"/>
-<junction x="-5.08" y="18.796"/>
 <pinref part="D5" gate="A" pin="A"/>
+<pinref part="U$13" gate="G$1" pin="E"/>
+<wire x1="88.9" y1="7.62" x2="78.74" y2="7.62" width="0.1524" layer="91"/>
+<junction x="78.74" y="7.62"/>
 </segment>
 </net>
@@
 <junction x="38.1" y="30.48"/>
 <pinref part="R3" gate="G$1" pin="2"/>
-<pinref part="U$12" gate="G$1" pin="+"/>
-<wire x1="15.24" y1="30.48" x2="5.08" y2="30.48" width="0.1524" layer="91"/>
 <junction x="15.24" y="30.48"/>
-<pinref part="U$11" gate="G$1" pin="+"/>
-<wire x1="5.08" y1="30.48" x2="-5.08" y2="30.48" width="0.1524" layer="91"/>
-<junction x="5.08" y="30.48"/>
+<wire x1="15.24" y1="30.48" x2="-12.7" y2="30.48" width="0.1524" layer="91"/>
 <wire x1="30.48" y1="45.72" x2="30.48" y2="30.48" width="0.1524" layer="91"/>
 <label x="38.1" y="45.72" size="1.778" layer="95"/>
-<wire x1="-5.08" y1="30.48" x2="-12.7" y2="30.48" width="0.1524" layer="91"/>
 <wire x1="-12.7" y1="30.48" x2="-12.7" y2="27.94" width="0.1524" layer="91"/>
-<junction x="-5.08" y="30.48"/>
 <pinref part="D5" gate="A" pin="K"/>
 </segment>

Commit message: add
Parts:
- added D4: (no value), zetex:DS_E2L
- added T1: S8050, transistor:2N3904
- added X1: 22-23-2021, con-molex:22-23-2021
Connections:
- new net N$1: D4.A, T1.B
- net CHARGE: now also T1.C
- net SWITCH: now also U$13.G
- net UC: now also D4.K
- net V-: now also T1.E
Other:
- moved on the sheet: D5
Changed lines of the file:
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@@
 <part name="D3" library="zetex" deviceset="DS_E2L" device="" package3d_urn="urn:adsk.eagle:package:30989/1" value="400v"/>
 <part name="U$13" library="untitled" deviceset="IGBT-N-TO247" device=""/>
+<part name="X1" library="con-molex" library_urn="urn:adsk.eagle:library:165" deviceset="22-23-2021" device="" package3d_urn="urn:adsk.eagle:package:8078633/1"/>
+<part name="D4" library="zetex" deviceset="DS_E2L" device="" package3d_urn="urn:adsk.eagle:package:30989/1"/>
+<part name="T1" library="transistor" library_urn="urn:adsk.eagle:library:402" deviceset="2N3904" device="" package3d_urn="urn:adsk.eagle:package:28523/2" value="S8050"/>
 </parts>
 <sheets>
@@
 <instance part="U$6" gate="G$1" x="83.82" y="25.4" smashed="yes" rot="R270"/>
 <instance part="D1" gate="1" x="73.66" y="22.86" smashed="yes" rot="R90"/>
-<instance part="U$9" gate="G$1" x="76.2" y="12.7" smashed="yes">
-<attribute name="VALUE" x="79.756" y="13.081" size="1.778" layer="96"/>
-</instance>
+<instance part="U$9" gate="G$1" x="76.2" y="12.7" smashed="yes"/>
 <instance part="D2" gate="1" x="25.4" y="45.72" smashed="yes">
 <attribute name="NAME" x="27.94" y="46.2026" size="1.778" layer="95"/>
@@
 <attribute name="VALUE" x="33.02" y="10.16" size="1.778" layer="96"/>
 </instance>
-<instance part="D5" gate="A" x="-12.7" y="25.4" smashed="yes" rot="R90">
-<attribute name="NAME" x="-13.335" y="27.94" size="1.778" layer="95" rot="R90"/>
-<attribute name="VALUE" x="-10.795" y="27.94" size="1.778" layer="96" rot="R90"/>
+<instance part="D5" gate="A" x="2.54" y="25.4" smashed="yes" rot="R90">
+<attribute name="NAME" x="1.905" y="27.94" size="1.778" layer="95" rot="R90"/>
+<attribute name="VALUE" x="4.445" y="27.94" size="1.778" layer="96" rot="R90"/>
 </instance>
 <instance part="D3" gate="A" x="5.08" y="68.58" smashed="yes" rot="R180">
@@
 <attribute name="VALUE" x="2.54" y="70.485" size="1.778" layer="96" rot="R180"/>
 </instance>
-<instance part="U$13" gate="G$1" x="86.36" y="12.7" smashed="yes">
-<attribute name="VALUE" x="89.916" y="13.081" size="1.778" layer="96"/>
+<instance part="U$13" gate="G$1" x="86.36" y="12.7" smashed="yes"/>
+<instance part="X1" gate="-1" x="137.16" y="38.1" smashed="yes">
+<attribute name="NAME" x="139.7" y="37.338" size="1.524" layer="95"/>
+<attribute name="VALUE" x="136.398" y="39.497" size="1.778" layer="96"/>
+</instance>
+<instance part="X1" gate="-2" x="137.16" y="35.56" smashed="yes">
+<attribute name="NAME" x="139.7" y="34.798" size="1.524" layer="95"/>
+</instance>
+<instance part="D4" gate="A" x="-7.62" y="30.48" smashed="yes">
+<attribute name="NAME" x="-5.08" y="31.115" size="1.778" layer="95"/>
+<attribute name="VALUE" x="-5.08" y="28.575" size="1.778" layer="96"/>
+</instance>
+<instance part="T1" gate="G1" x="-7.62" y="17.78" smashed="yes">
+<attribute name="NAME" x="-10.16" y="20.32" size="1.778" layer="95"/>
+<attribute name="VALUE" x="-7.62" y="17.78" size="1.778" layer="96"/>
 </instance>
 </instances>
@@
 <segment>
 <pinref part="U$9" gate="G$1" pin="G"/>
-<wire x1="71.12" y1="10.16" x2="66.04" y2="10.16" width="0.1524" layer="91"/>
+<wire x1="71.12" y1="10.16" x2="68.58" y2="10.16" width="0.1524" layer="91"/>
 <label x="66.04" y="10.16" size="1.778" layer="95"/>
+<pinref part="U$13" gate="G$1" pin="G"/>
+<wire x1="68.58" y1="10.16" x2="66.04" y2="10.16" width="0.1524" layer="91"/>
+<wire x1="81.28" y1="10.16" x2="81.28" y2="12.7" width="0.1524" layer="91"/>
+<wire x1="81.28" y1="12.7" x2="68.58" y2="12.7" width="0.1524" layer="91"/>
+<wire x1="68.58" y1="12.7" x2="68.58" y2="10.16" width="0.1524" layer="91"/>
+<junction x="68.58" y="10.16"/>
 </segment>
 </net>
@@
 <junction x="5.08" y="5.08"/>
 <pinref part="Q1" gate="G$1" pin="S"/>
+<pinref part="T1" gate="G1" pin="E"/>
+<wire x1="-5.08" y1="12.7" x2="5.08" y2="12.7" width="0.1524" layer="91"/>
+<wire x1="5.08" y1="12.7" x2="5.08" y2="5.08" width="0.1524" layer="91"/>
 </segment>
 <segment>
@@
 <wire x1="76.2" y1="85.344" x2="71.12" y2="85.344" width="0.1524" layer="91"/>
 </segment>
+<segment>
+<pinref part="T1" gate="G1" pin="C"/>
+<wire x1="-5.08" y1="22.86" x2="-5.08" y2="25.4" width="0.1524" layer="91"/>
+<label x="-10.16" y="25.4" size="1.778" layer="95"/>
+</segment>
 </net>
 <net name="N$10" class="0">
 <segment>
-<wire x1="-12.7" y1="18.796" x2="15.24" y2="18.796" width="0.1524" layer="91"/>
+<wire x1="2.54" y1="18.796" x2="15.24" y2="18.796" width="0.1524" layer="91"/>
 <pinref part="U$4" gate="G$1" pin="-"/>
 <pinref part="R3" gate="G$1" pin="1"/>
@@
 <junction x="15.24" y="18.796"/>
 <pinref part="Q1" gate="G$1" pin="D"/>
-<wire x1="-12.7" y1="22.86" x2="-12.7" y2="18.796" width="0.1524" layer="91"/>
+<wire x1="2.54" y1="22.86" x2="2.54" y2="18.796" width="0.1524" layer="91"/>
 <pinref part="D5" gate="A" pin="A"/>
 <pinref part="U$13" gate="G$1" pin="E"/>
-<wire x1="88.9" y1="7.62" x2="78.74" y2="7.62" width="0.1524" layer="91"/>
-<junction x="78.74" y="7.62"/>
+<wire x1="88.9" y1="7.62" x2="88.9" y2="5.08" width="0.1524" layer="91"/>
+<wire x1="88.9" y1="5.08" x2="78.74" y2="5.08" width="0.1524" layer="91"/>
+<junction x="78.74" y="5.08"/>
 </segment>
 </net>
@@
 <pinref part="R3" gate="G$1" pin="2"/>
 <junction x="15.24" y="30.48"/>
-<wire x1="15.24" y1="30.48" x2="-12.7" y2="30.48" width="0.1524" layer="91"/>
+<wire x1="15.24" y1="30.48" x2="2.54" y2="30.48" width="0.1524" layer="91"/>
 <wire x1="30.48" y1="45.72" x2="30.48" y2="30.48" width="0.1524" layer="91"/>
 <label x="38.1" y="45.72" size="1.778" layer="95"/>
-<wire x1="-12.7" y1="30.48" x2="-12.7" y2="27.94" width="0.1524" layer="91"/>
+<wire x1="2.54" y1="30.48" x2="2.54" y2="27.94" width="0.1524" layer="91"/>
 <pinref part="D5" gate="A" pin="K"/>
-</segment>
-</net>
+<pinref part="D4" gate="A" pin="K"/>
+<wire x1="2.54" y1="30.48" x2="-5.08" y2="30.48" width="0.1524" layer="91"/>
+<junction x="2.54" y="30.48"/>
+</segment>
+</net>
+<net name="N$1" class="0">
+<segment>
+<pinref part="D4" gate="A" pin="A"/>
+<wire x1="-10.16" y1="30.48" x2="-15.24" y2="30.48" width="0.1524" layer="91"/>
+<pinref part="T1" gate="G1" pin="B"/>
+<wire x1="-15.24" y1="30.48" x2="-15.24" y2="17.78" width="0.1524" layer="91"/>
+<wire x1="-15.24" y1="17.78" x2="-10.16" y2="17.78" width="0.1524" layer="91"/>
+</segment>
+</net>

Commit message: add
Parts:
- removed X1: 22-23-2021, con-molex:22-23-2021
- added J1: 61300311121, Headers:61300311121

Commit message: add
Parts:
- added OK2: SFH618A-3, optocoupler:SFH618A-3
- added Q2: 2N3906, transistor-pnp:2N3906
- added R10, R6, R7, R8, R9: 10k, rcl:R-EU_0207/2V
- added T3: s8050, transistor:2N3704
Connections:
- removed net N$7: BT+.MOUNT, OK1.EMIT, R1.1, R4.1
- new net BT+: BT+.MOUNT, OK1.COL, OK2.COL, R1.1, R4.1, R6.1
- new net N$11: J1.1, OK2.A
- new net N$12: OK2.EMIT, Q2.B, R8.1, T3.B
- new net N$13: Q2.C, R7.1
- new net N$14: R6.2, T3.C
- new net N$8: Q2.E, R9.1, T3.E
- new net V2-: J1.2, OK2.C
- net N$10: now also R10.1
- net N$5: now also OK1.EMIT; no longer OK1.COL
- net SWITCH: now also R10.2, R9.2
- net V-: now also R7.2, R8.2
Other:
- moved on the sheet: BT+, BT-, J1, R1, R2, R4, R5
