File: upvol.sch (EAGLE design)
At the start: 11 parts, among them IC1 LM393D, J1 61300311121, J2 61300211121

Commit message: add
Parts:
- removed J2: 61300211121, Headers:61300211121
- added T1: s9014, transistor:-NPN-SOT23-EBC
- R1, R2, R4: device OPL_Resistor:DIP-RES-10K-5%-1/4W(PR-D2.3XL6.5MM) -> 52101-101-REV-A_v16:RC-MASTER-SMD_R_0603MP
- R3: value 100 -> 4.7k; device OPL_Resistor:DIP-RES-10K-5%-1/4W(PR-D2.3XL6.5MM) -> 52101-101-REV-A_v16:RC-MASTER-SMD_R_0603MP
Connections:
- new net N$5: IC1A.OUT, T1.B
- net N$1: now also C1.2, U$1.C; no longer C1.1, U$1.E
- net OUT: now also T1.C; no longer IC1A.OUT
- net V+: now also IC1P.V+; no longer J2.2
- net V-: now also C1.1, IC1P.V-, T1.E, U$1.E; no longer C1.2, J2.1, U$1.C
Other:
- moved on the sheet: C1, IC1A, J1, LED1, U$1

Commit message: 更新输入模块
Parts:
- R1: device 52101-101-REV-A_v16:RC-MASTER-SMD_R_0603MP -> rcl:R-EU_0204/2V
Changed lines of the file:
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@@
 <?xml version="1.0" encoding="utf-8"?>
 <!DOCTYPE eagle SYSTEM "eagle.dtd">
-<eagle version="9.6.2">
+<eagle version="9.5.1">
 <drawing>
 <settings>
@@
 <parts>
 <part name="IC1" library="linear" library_urn="urn:adsk.eagle:library:262" deviceset="LM393" device="D" package3d_urn="urn:adsk.eagle:package:16404/2"/>
-<part name="R1" library="52101-101-REV-A_v16" library_urn="urn:adsk.eagle:library:21899384" deviceset="RC-MASTER-SMD_R_" device="0603MP" package3d_urn="urn:adsk.eagle:package:15662272/2" value="10K"/>
+<part name="R1" library="rcl" library_urn="urn:adsk.eagle:library:334" deviceset="R-EU_" device="0204/2V" package3d_urn="urn:adsk.eagle:package:23495/1" value="10K"/>
 <part name="R2" library="52101-101-REV-A_v16" library_urn="urn:adsk.eagle:library:21899384" deviceset="RC-MASTER-SMD_R_" device="0603MP" package3d_urn="urn:adsk.eagle:package:15662272/2" value="10K"/>
 <part name="R3" library="52101-101-REV-A_v16" library_urn="urn:adsk.eagle:library:21899384" deviceset="RC-MASTER-SMD_R_" device="0603MP" package3d_urn="urn:adsk.eagle:package:15662272/2" value="4.7k"/>
@@
 packages will not be understood (or retained) with this version.
 </note>
+<note version="8.4" severity="warning">
+Since Version 8.4, EAGLE supports properties for SPICE simulation.
+Probes in schematics and SPICE mapping objects found in parts and library devices
+will not be understood with this version. Update EAGLE to the latest version
+for full support of SPICE simulation.
+</note>
 </compatibility>
